File: input.kicad_sch (KiCad schematic)
At the start: 22 parts, among them U1 TPS5430DDAR, U6 AMS1117-3.3

Commit message: begin layout
Parts:
- C11, C12, C13, C14, C15, C16, C17, C18, C4, C5, C6, C7, C8, C9: footprint PCM_Capacitor_SMD_AKL:C_0402_1005Metric -> PCM_Capacitor_SMD_AKL:C_0603_1608Metric
- R10, R11: footprint PCM_Resistor_SMD_AKL:R_0402_1005Metric -> PCM_Resistor_SMD_AKL:R_0603_1608Metric
Changed lines of the file:
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@@
 			)
 		)
-		(property "Footprint" "PCM_Capacitor_SMD_AKL:C_0402_1005Metric"
+		(property "Footprint" "PCM_Capacitor_SMD_AKL:C_0603_1608Metric"
 			(at 242.57 87.63 0)
 			(effects
@@
 			)
 		)
-		(property "Footprint" "PCM_Capacitor_SMD_AKL:C_0402_1005Metric"
+		(property "Footprint" "PCM_Capacitor_SMD_AKL:C_0603_1608Metric"
 			(at 219.71 87.63 0)
 			(effects
@@
 			)
 		)
-		(property "Footprint" "PCM_Capacitor_SMD_AKL:C_0402_1005Metric"
+		(property "Footprint" "PCM_Capacitor_SMD_AKL:C_0603_1608Metric"
 			(at 76.2 85.09 0)
 			(effects
@@
 			)
 		)
-		(property "Footprint" "PCM_Capacitor_SMD_AKL:C_0402_1005Metric"
+		(property "Footprint" "PCM_Capacitor_SMD_AKL:C_0603_1608Metric"
 			(at 143.51 78.74 0)
 			(effects
@@
 			)
 		)
-		(property "Footprint" "PCM_Capacitor_SMD_AKL:C_0402_1005Metric"
+		(property "Footprint" "PCM_Capacitor_SMD_AKL:C_0603_1608Metric"
 			(at 212.09 87.63 0)
 			(effects
@@
 			)
 		)
-		(property "Footprint" "PCM_Capacitor_SMD_AKL:C_0402_1005Metric"
+		(property "Footprint" "PCM_Capacitor_SMD_AKL:C_0603_1608Metric"
 			(at 246.38 87.63 0)
 			(effects
@@
 			)
 		)
-		(property "Footprint" "PCM_Capacitor_SMD_AKL:C_0402_1005Metric"
+		(property "Footprint" "PCM_Capacitor_SMD_AKL:C_0603_1608Metric"
 			(at 208.28 87.63 0)
 			(effects
@@
 			)
 		)
-		(property "Footprint" "PCM_Resistor_SMD_AKL:R_0402_1005Metric"
+		(property "Footprint" "PCM_Resistor_SMD_AKL:R_0603_1608Metric"
 			(at 170.18 71.12 0)
 			(effects
@@
 			)
 		)
-		(property "Footprint" "PCM_Capacitor_SMD_AKL:C_0402_1005Metric"
+		(property "Footprint" "PCM_Capacitor_SMD_AKL:C_0603_1608Metric"
 			(at 204.47 87.63 0)
 			(effects
@@
 			)
 		)
-		(property "Footprint" "PCM_Capacitor_SMD_AKL:C_0402_1005Metric"
+		(property "Footprint" "PCM_Capacitor_SMD_AKL:C_0603_1608Metric"
 			(at 83.82 85.09 0)
 			(effects
@@
 			)
 		)
-		(property "Footprint" "PCM_Capacitor_SMD_AKL:C_0402_1005Metric"
+		(property "Footprint" "PCM_Capacitor_SMD_AKL:C_0603_1608Metric"
 			(at 72.39 85.09 0)
 			(effects
@@
 			)
 		)
-		(property "Footprint" "PCM_Capacitor_SMD_AKL:C_0402_1005Metric"
+		(property "Footprint" "PCM_Capacitor_SMD_AKL:C_0603_1608Metric"
 			(at 80.01 85.09 0)
 			(effects
@@
 			)
 		)
-		(property "Footprint" "PCM_Resistor_SMD_AKL:R_0402_1005Metric"
+		(property "Footprint" "PCM_Resistor_SMD_AKL:R_0603_1608Metric"
 			(at 170.18 78.74 0)
 			(effects
@@
 			)
 		)
-		(property "Footprint" "PCM_Capacitor_SMD_AKL:C_0402_1005Metric"
+		(property "Footprint" "PCM_Capacitor_SMD_AKL:C_0603_1608Metric"
 			(at 250.19 87.63 0)
 			(effects
@@
 			)
 		)
-		(property "Footprint" "PCM_Capacitor_SMD_AKL:C_0402_1005Metric"
+		(property "Footprint" "PCM_Capacitor_SMD_AKL:C_0603_1608Metric"
 			(at 68.58 85.09 0)
 			(effects
@@
 			)
 		)
-		(property "Footprint" "PCM_Capacitor_SMD_AKL:C_0402_1005Metric"
+		(property "Footprint" "PCM_Capacitor_SMD_AKL:C_0603_1608Metric"
 			(at 215.9 87.63 0)
 			(effects

Commit message: add cubemx project and redo some layour with new parts
Parts:
- renumbered C3 to C15, C4 to C16, C5 to C17, C6 to C18, C7 to C19, C8 to C20, C9 to C21, C10 to C22, C11 to C23, C12 to C24, C13 to C25, C14 to C26, C15 to C27, C16 to C28, C17 to C29, C18 to C30, D2 to D3, R10 to R7, R11 to R8, U1 to U10, U6 to U11
Changed lines of the file:
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@@
 		(on_board yes)
 		(dnp no)
-		(property "Reference" "#PWR04"
+		(property "Reference" "#PWR043"
 			(at 83.82 97.79 0)
 			(effects
@@
 			(project "Active-Dampers"
 				(path "/81892b73-0b2d-4185-94d6-5966c81d614d/037f147e-6821-4821-9a3a-0a44cbef2c0e"
-					(reference "#PWR04")
+					(reference "#PWR043")
 					(unit 1)
 				)
@@
 		(on_board yes)
 		(dnp no)
-		(property "Reference" "C16"
+		(property "Reference" "C28"
 			(at 241.3 82.55 90)
 			(effects
@@
 			(project "Active-Dampers"
 				(path "/81892b73-0b2d-4185-94d6-5966c81d614d/037f147e-6821-4821-9a3a-0a44cbef2c0e"
-					(reference "C16")
+					(reference "C28")
 					(unit 1)
 				)
@@
 		(dnp no)
 		(fields_autoplaced yes)
-		(property "Reference" "U1"
+		(property "Reference" "U10"
 			(at 123.19 71.12 0)
 			(effects
@@
 			(project "Active-Dampers"
 				(path "/81892b73-0b2d-4185-94d6-5966c81d614d/037f147e-6821-4821-9a3a-0a44cbef2c0e"
-					(reference "U1")
+					(reference "U10")
 					(unit 1)
 				)
@@
 		(on_board yes)
 		(dnp no)
-		(property "Reference" "C15"
+		(property "Reference" "C27"
 			(at 218.44 82.55 90)
 			(effects
@@
 			(project "Active-Dampers"
 				(path "/81892b73-0b2d-4185-94d6-5966c81d614d/037f147e-6821-4821-9a3a-0a44cbef2c0e"
-					(reference "C15")
+					(reference "C27")
 					(unit 1)
 				)
@@
 		(on_board yes)
 		(dnp no)
-		(property "Reference" "C6"
+		(property "Reference" "C18"
 			(at 74.93 80.01 90)
 			(effects
@@
 			(project "Active-Dampers"
 				(path "/81892b73-0b2d-4185-94d6-5966c81d614d/037f147e-6821-4821-9a3a-0a44cbef2c0e"
-					(reference "C6")
+					(reference "C18")
 					(unit 1)
 				)
@@
 		(on_board yes)
 		(dnp no)
-		(property "Reference" "C3"
+		(property "Reference" "C15"
 			(at 67.31 82.9309 0)
 			(effects
@@
 			(project "Active-Dampers"
 				(path "/81892b73-0b2d-4185-94d6-5966c81d614d/037f147e-6821-4821-9a3a-0a44cbef2c0e"
-					(reference "C3")
+					(reference "C15")
 					(unit 1)
 				)
@@
 		(on_board yes)
 		(dnp no)
-		(property "Reference" "#PWR045"
+		(property "Reference" "#PWR046"
 			(at 161.29 97.79 0)
 			(effects
@@
 			(project "Active-Dampers"
 				(path "/81892b73-0b2d-4185-94d6-5966c81d614d/037f147e-6821-4821-9a3a-0a44cbef2c0e"
-					(reference "#PWR045")
+					(reference "#PWR046")
 					(unit 1)
 				)
@@
 		(on_board yes)
 		(dnp no)
-		(property "Reference" "C9"
+		(property "Reference" "C21"
 			(at 148.59 77.47 90)
 			(effects
@@
 			(project "Active-Dampers"
 				(path "/81892b73-0b2d-4185-94d6-5966c81d614d/037f147e-6821-4821-9a3a-0a44cbef2c0e"
-					(reference "C9")
+					(reference "C21")
 					(unit 1)
 				)
@@
 		(on_board yes)
 		(dnp no)
-		(property "Reference" "C13"
+		(property "Reference" "C25"
 			(at 210.82 82.55 90)
 			(effects
@@
 			(project "Active-Dampers"
 				(path "/81892b73-0b2d-4185-94d6-5966c81d614d/037f147e-6821-4821-9a3a-0a44cbef2c0e"
-					(reference "C13")
+					(reference "C25")
 					(unit 1)
 				)
@@
 		(on_board yes)
 		(dnp no)
-		(property "Reference" "C17"
+		(property "Reference" "C29"
 			(at 245.11 82.55 90)
 			(effects
@@
 			(project "Active-Dampers"
 				(path "/81892b73-0b2d-4185-94d6-5966c81d614d/037f147e-6821-4821-9a3a-0a44cbef2c0e"
-					(reference "C17")
+					(reference "C29")
 					(unit 1)
 				)
@@
 		(on_board yes)
 		(dnp no)
-		(property "Reference" "#PWR043"
+		(property "Reference" "#PWR044"
 			(at 120.65 97.79 0)
 			(effects
@@
 			(project "Active-Dampers"
 				(path "/81892b73-0b2d-4185-94d6-5966c81d614d/037f147e-6821-4821-9a3a-0a44cbef2c0e"
-					(reference "#PWR043")
+					(reference "#PWR044")
 					(unit 1)
 				)
@@
 		(on_board yes)
 		(dnp no)
-		(property "Reference" "C12"
+		(property "Reference" "C24"
 			(at 207.01 82.55 90)
 			(effects
@@
 			(project "Active-Dampers"
 				(path "/81892b73-0b2d-4185-94d6-5966c81d614d/037f147e-6821-4821-9a3a-0a44cbef2c0e"
-					(reference "C12")
+					(reference "C24")
 					(unit 1)
 				)
@@
 		(on_board yes)
 		(dnp no)
-		(property "Reference" "C10"
+		(property "Reference" "C22"
 			(at 165.1 82.9309 0)
 			(effects
@@
 			(project "Active-Dampers"
 				(path "/81892b73-0b2d-4185-94d6-5966c81d614d/037f147e-6821-4821-9a3a-0a44cbef2c0e"
-					(reference "C10")
+					(reference "C22")
 					(unit 1)
 				)
@@
 		(on_board yes)
 		(dnp no)
-		(property "Reference" "#PWR046"
+		(property "Reference" "#PWR047"
 			(at 170.18 100.33 0)
 			(effects
@@
 			(project "Active-Dampers"
 				(path "/81892b73-0b2d-4185-94d6-5966c81d614d/037f147e-6821-4821-9a3a-0a44cbef2c0e"
-					(reference "#PWR046")
+					(reference "#PWR047")
 					(unit 1)
 				)
@@
 		(on_board yes)
 		(dnp no)
-		(property "Reference" "R10"
+		(property "Reference" "R7"
 			(at 167.64 82.55 90)
 			(effects
@@
 			)
 		)
+		(property "Sim.Device" ""
+			(at 170.18 82.55 0)
+			(effects
+				(font
+					(size 1.27 1.27)
+				)
+				(hide yes)
+			)
+		)
+		(property "Sim.Pins" ""
+			(at 170.18 82.55 0)
+			(effects
+				(font
+					(size 1.27 1.27)
+				)
+				(hide yes)
+			)
+		)
 		(pin "1"
 		)
@@
 			(project "Active-Dampers"
 				(path "/81892b73-0b2d-4185-94d6-5966c81d614d/037f147e-6821-4821-9a3a-0a44cbef2c0e"
-					(reference "R10")
+					(reference "R7")
 					(unit 1)
 				)
@@
 		(dnp no)
 		(fields_autoplaced yes)
-		(property "Reference" "U6"
+		(property "Reference" "U11"
 			(at 231.14 72.39 0)
 			(effects
@@
 			(project "Active-Dampers"
 				(path "/81892b73-0b2d-4185-94d6-5966c81d614d/037f147e-6821-4821-9a3a-0a44cbef2c0e"
-					(reference "U6")
+					(reference "U11")
 					(unit 1)
 				)
@@
 		(on_board yes)
 		(dnp no)
-		(property "Reference" "#PWR05"
+		(property "Reference" "#PWR048"
 			(at 250.19 102.87 0)
 			(effects
@@
 			(project "Active-Dampers"
 				(path "/81892b73-0b2d-4185-94d6-5966c81d614d/037f147e-6821-4821-9a3a-0a44cbef2c0e"
-					(reference "#PWR05")
+					(reference "#PWR048")
 					(unit 1)
 				)
@@
 		(on_board yes)
 		(dnp no)
-		(property "Reference" "C11"
+		(property "Reference" "C23"
 			(at 203.2 82.55 90)
 			(effects
@@
 			(project "Active-Dampers"
 				(path "/81892b73-0b2d-4185-94d6-5966c81d614d/037f147e-6821-4821-9a3a-0a44cbef2c0e"
-					(reference "C11")
+					(reference "C23")
 					(unit 1)
 				)
@@
 		(on_board yes)
 		(dnp no)
-		(property "Reference" "C8"
+		(property "Reference" "C20"
 			(at 82.55 80.01 90)
 			(effects
@@
 			(project "Active-Dampers"
 				(path "/81892b73-0b2d-4185-94d6-5966c81d614d/037f147e-6821-4821-9a3a-0a44cbef2c0e"
-					(reference "C8")
+					(reference "C20")
 					(unit 1)
 				)
@@
 		(dnp no)
 		(fields_autoplaced yes)
-		(property "Reference" "D2"
+		(property "Reference" "D3"
 			(at 153.67 80.9624 0)
 			(effects
@@
 			(project "Active-Dampers"
 				(path "/81892b73-0b2d-4185-94d6-5966c81d614d/037f147e-6821-4821-9a3a-0a44cbef2c0e"
-					(reference "D2")
+					(reference "D3")
 					(unit 1)
 				)
@@
 		(on_board yes)
 		(dnp no)
-		(property "Reference" "C5"
+		(property "Reference" "C17"
 			(at 71.12 80.01 90)
 			(effects
@@
 			(project "Active-Dampers"
 				(path "/81892b73-0b2d-4185-94d6-5966c81d614d/037f147e-6821-4821-9a3a-0a44cbef2c0e"
-					(reference "C5")
+					(reference "C17")
 					(unit 1)
 				)
@@
 		(on_board yes)
 		(dnp no)
-		(property "Reference" "C7"
+		(property "Reference" "C19"
 			(at 78.74 80.01 90)
 			(effects
@@
 			(project "Active-Dampers"
 				(path "/81892b73-0b2d-4185-94d6-5966c81d614d/037f147e-6821-4821-9a3a-0a44cbef2c0e"
-					(reference "C7")
+					(reference "C19")
 					(unit 1)
 				)
@@
 		(on_board yes)
 		(dnp no)
-		(property "Reference" "R11"
+		(property "Reference" "R8"
 			(at 167.64 90.17 90)
 			(effects
@@
 			)
 		)
+		(property "Sim.Device" ""
+			(at 170.18 90.17 0)
+			(effects
+				(font
+					(size 1.27 1.27)
+				)
+				(hide yes)
+			)
+		)
+		(property "Sim.Pins" ""
+			(at 170.18 90.17 0)
+			(effects
+				(font
+					(size 1.27 1.27)
+				)
+				(hide yes)
+			)
+		)
 		(pin "1"
 		)
@@
 			(project "Active-Dampers"
 				(path "/81892b73-0b2d-4185-94d6-5966c81d614d/037f147e-6821-4821-9a3a-0a44cbef2c0e"
-					(reference "R11")
+					(reference "R8")
 					(unit 1)
 				)
@@
 		(on_board yes)
 		(dnp no)
-		(property "Reference" "C18"
+		(property "Reference" "C30"
 			(at 248.92 82.55 90)
 			(effects
@@
 			(project "Active-Dampers"
 				(path "/81892b73-0b2d-4185-94d6-5966c81d614d/037f147e-6821-4821-9a3a-0a44cbef2c0e"
-					(reference "C18")
+					(reference "C30")
 					(unit 1)
 				)
@@
 		(on_board yes)
 		(dnp no)
-		(property "Reference" "#PWR044"
+		(property "Reference" "#PWR045"
 			(at 151.13 92.71 0)
 			(effects
@@
 			(project "Active-Dampers"
 				(path "/81892b73-0b2d-4185-94d6-5966c81d614d/037f147e-6821-4821-9a3a-0a44cbef2c0e"
-					(reference "#PWR044")
+					(reference "#PWR045")
 					(unit 1)
 				)
@@
 		(on_board yes)
 		(dnp no)
-		(property "Reference" "C4"
+		(property "Reference" "C16"
 			(at 67.31 80.01 90)
 			(effects
@@
 			(project "Active-Dampers"
 				(path "/81892b73-0b2d-4185-94d6-5966c81d614d/037f147e-6821-4821-9a3a-0a44cbef2c0e"
-					(reference "C4")
+					(reference "C16")
 					(unit 1)
 				)
@@
 		(on_board yes)
 		(dnp no)
-		(property "Reference" "C14"
+		(property "Reference" "C26"
 			(at 214.63 82.55 90)
 			(effects
@@
 			(project "Active-Dampers"
 				(path "/81892b73-0b2d-4185-94d6-5966c81d614d/037f147e-6821-4821-9a3a-0a44cbef2c0e"
-					(reference "C14")
+					(reference "C26")
 					(unit 1)
 				)
