File: Active-Dampers.kicad_sch (KiCad schematic)
At the start: 48 parts, among them J1 Conn_ARM_JTAG_SWD_10, J2 FL, J3 FR, J4 RL, J5 RR, J6 Barrel_Jack_Switch_Pin3Ring, J7 USB_C_Receptacle_USB2.0_16P, J8 OLED, SW1 SW_SPST, U1 MPU-6050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

Commit message: prod
Parts:
- C1, C34, C6: LCSC (none) -> C14663
- C10: LCSC (none) -> C1604
- C11, C12, C13, C14: LCSC (none) -> C23630
- C2, C3: LCSC (none) -> C1653
- C5, C8, C9: LCSC (none) -> C96446
- C7: LCSC (none) -> C15849
- D12, D14, D7: LCSC (none) -> C2286
- J1: footprint Manual_Parts:CNC_3220-10-0300-00 -> SamacSys_Parts:62701021621; Manufacturer_Part_Number CNC_3220-10-0300-00 -> (none); now left out of the parts list
- J2, J3, J4, J5, J6, J8: now left out of the parts list
- J7: LCSC (none) -> C165948
- R1: LCSC (none) -> C21190
- R13: LCSC (none) -> C23138
- R16, R5: footprint PCM_Resistor_SMD_AKL:R_0402_1005Metric -> PCM_Resistor_SMD_AKL:R_0603_1608Metric; LCSC (none) -> C23162
- R2: LCSC (none) -> C25804
- R28: LCSC (none) -> C23228
- R3, R4: LCSC (none) -> C23186
- R30: LCSC (none) -> C22975
- SW1: LCSC (none) -> C720477
- U1: LCSC (none) -> C24112
- U6, U7, U8, U9: LCSC (none) -> C131079
Connections:
- net AIN2_FR: now also U2.27 (PB14)
- net BIN2_FR: now also U2.26 (PB13)
- net GND: now also U1.1 (CLKIN), U1.18 (GND), U1.9 (AD0)
- net IMU_INT: now also U2.41 (PB5)
- net SCL: now also U2.42 (PB6)
- net SDA: now also U2.43 (PB7)
