File: Active-Dampers.kicad_pcb (KiCad board)
At the start: 4 copper layers, 50 x 50 mm, 70 parts, among them J1 Conn_ARM_JTAG_SWD_10, J2 FL, J3 FR, J4 RL, J5 RR, J6 Barrel_Jack_Switch_Pin3Ring, J7 USB_C_Receptacle_USB2.0_16P, J8 OLED, SW1 SW_SPST, U1 MPU-6050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

Commit message: create prod files
Parts:
- J2, J3, J4, J5: footprint Connector_JST:JST_XH_B4B-XH-AM_1x04_P2.50mm_Vertical -> Connector_JST:JST_XH_B4B-XH-A_1x04_P2.50mm_Vertical
