File: Master/Active-Damper-Master.kicad_pcb (KiCad board)
At the start: 2 copper layers, 50 x 55 mm, 75 parts, among them IC1 ESP32-C6-WROOM-1-N8, J1 Conn_01x07, J2 PINHD_1x2_Male, J3 PINHD_1x2_Male, J6 USB_C_Receptacle_USB2.0_16P, SW2 SW_SPST, SW3 SW_SPST, U1 SN65HVD230, U2 TPS5430DDAR, U3 AMS1117-3.3, U4 SN65HVD230, U5 LSM6DS3

Commit message: finish prod files for master
Parts:
- removed D4, D5: LED BLUE, PCM_LED_SMD_AKL:LED_0603_1608Metric
- removed J1: Conn_01x07, Connector_JST:JST_XH_S7B-XH-A-1_1x07_P2.50mm_Horizontal
- removed J2, J3: PINHD_1x2_Male, Connector_PinHeader_2.54mm:PinHeader_1x02_P2.54mm_Vertical
- removed R24: 1k, PCM_Resistor_SMD_AKL:R_0603_1608Metric
- removed R4: 680, PCM_Resistor_SMD_AKL:R_0603_1608Metric
- removed R5: 330, PCM_Resistor_SMD_AKL:R_0603_1608Metric
- removed R52: 4.7k, PCM_Capacitor_SMD_AKL:C_0603_1608Metric
- removed U1: SN65HVD230, Package_SO:SOIC-8_3.9x4.9mm_P1.27mm
- removed U5: LSM6DS3, Package_LGA:LGA-14_3x2.5mm_P0.5mm_LayoutBorder3x4y
- added D10: SS54, PCM_JLCPCB:D_SMA, F.Cu at (162.2, 114.5)
- added J7: POWER, Connector_JST:JST_XH_S3B-XH-A-1_1x03_P2.50mm_Horizontal, F.Cu at (158.5, 120.9)
- added J8: CAN_2, Connector_JST:JST_XH_S3B-XH-A-1_1x03_P2.50mm_Horizontal, F.Cu at (147.5, 120.9)
- added J9: CAN_1, Connector_JST:JST_XH_S3B-XH-A-1_1x03_P2.50mm_Horizontal, F.Cu at (136.5, 120.9)
- added JP2: SolderJumper_2_Open, Jumper:SolderJumper-2_P1.3mm_Open_RoundedPad1.0x1.5mm, F.Cu at (140.0, 106.0)
- added JP4: SolderJumper_2_Open, Jumper:SolderJumper-2_P1.3mm_Open_RoundedPad1.0x1.5mm, F.Cu at (128.2, 106.2)
- added JP5: SolderJumper_3_Open, Jumper:SolderJumper-3_P1.3mm_Open_RoundedPad1.0x1.5mm, F.Cu at (171.6, 89.2)
- added Q1: AO3401A, Package_TO_SOT_SMD:SOT-23, F.Cu at (171.5, 82.2)
- added R53: 4.7k, PCM_Resistor_SMD_AKL:R_0603_1608Metric, F.Cu at (131.0, 82.2)
- added R54: 4.7k, PCM_Resistor_SMD_AKL:R_0603_1608Metric, F.Cu at (136.8, 88.0)
- added U6: TJA1051T, Package_SO:SOIC-8_3.9x4.9mm_P1.27mm, F.Cu at (133.0, 106.0)
- added U7: TJA1051T, Package_SO:SOIC-8_3.9x4.9mm_P1.27mm, F.Cu at (144.8, 106.0)
- R51: footprint PCM_Capacitor_SMD_AKL:C_0603_1608Metric -> PCM_Resistor_SMD_AKL:R_0603_1608Metric
- U4: value SN65HVD230 -> LIS3DH; footprint Package_SO:SOIC-8_3.9x4.9mm_P1.27mm -> Package_LGA:LGA-16_3x3mm_P0.5mm_LayoutBorder3x5y
- moved D7 34.0 mm to (168.2, 117.4)
- moved R9 30.6 mm to (168.2, 119.2), turned to 0 degrees
- moved U4 28.6 mm to (128.2, 82.5), turned to 90 degrees
- moved C3 7.15 mm to (168.3, 111.8)
- moved R51 6.63 mm to (136.8, 86.2), turned to 0 degrees
- moved C54 4.26 mm to (128.0, 113.5), turned to -90 degrees
- moved R46 4.24 mm to (131.2, 110.8), turned to 0 degrees
- moved R6 4.18 mm to (128.5, 98.5)
- moved L1 4.00 mm to (161.2, 107.7)
- moved R7 2.82 mm to (132.0, 98.5), turned to 0 degrees
- moved C11 1.50 mm to (153.5, 114.5)
- moved C12 1.50 mm to (155.5, 114.5)
- moved C13 1.50 mm to (151.5, 114.5)
- moved C14 1.50 mm to (149.5, 114.5)
- moved C15 1.50 mm to (157.5, 114.5)
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Connections:
- C3 pad 1: +12V -> Net-(JP5-B)
- C4 pad 2: +12V -> Net-(JP5-B)
- C48 pad 1: GND -> Net-(Q1-D)
- C5 pad 2: +12V -> Net-(JP5-B)
- C6 pad 2: +12V -> Net-(JP5-B)
- C7 pad 2: +12V -> Net-(JP5-B)
- C8 pad 2: +12V -> Net-(JP5-B)
- IC1 pad 24: unconnected-(IC1-RXD0-Pad24) -> /BATT_MEAS_ENA
- R8 pad 2: GND -> Net-(Q1-D)
- U2 pad 5: +12V -> Net-(JP5-C)
- U2 pad 7: +12V -> Net-(JP5-B)
- U4 pad 1: /RXD_2 -> +3.3V
- U4 pad 2: GND -> unconnected-(U4-NC-Pad2)
- U4 pad 3: +3.3V -> unconnected-(U4-NC-Pad3)
- U4 pad 4: /TXD_2 -> /SCL
- U4 pad 5: unconnected-(U4-Vref-Pad5) -> GND
- U4 pad 6: /CANL_2 -> /SDA
- U4 pad 7: /CANH_2 -> GND
- U4 pad 8: /Rs_2 -> Net-(U4-CS)
Routing:
- net Net-(JP5-B): track 0.00 -> 42.8 mm, vias 0 -> 6
- net +12V: track 19.8 -> 55.4 mm, vias 8 -> 1
- net /Rs_1: track 0.00 -> 31.4 mm, vias 0 -> 2
- net /RXD_1: track 0.00 -> 27.7 mm, vias 0 -> 2
- net /TXD_1: track 0.00 -> 24.9 mm, vias 0 -> 2
- net /SDA: track 0.00 -> 19.3 mm, vias 0 -> 2
- net /CANL_1: track 0.00 -> 19.1 mm, vias 0 -> 1
- net /SCL: track 0.00 -> 18.6 mm, vias 0 -> 2
- net /CANH_1: track 0.00 -> 17.6 mm, vias 0 -> 1
- net /USB+: track 0.00 -> 15.8 mm, vias 0 -> 2
- net Net-(Q1-D): track 0.00 -> 14.9 mm, vias 0 -> 2
- net +3.3V: track 6.17 -> 18.7 mm, vias 13 -> 21
- net /BATT_MEAS_ENA: track 0.00 -> 12.0 mm, vias 0 -> 2
- net /USB-: track 0.00 -> 11.7 mm
- net Net-(J6-CC1): track 0.00 -> 11.3 mm, vias 0 -> 2
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- removed copper zone on B.Cu, net +12V
Other:
- board text added: "CAN1"
- board text added: "CAN2"
- board text added: "PWR"

Commit message: add prod files, not done
Parts:
- removed J7: POWER, Connector_JST:JST_XH_S3B-XH-A-1_1x03_P2.50mm_Horizontal
- removed J8: CAN_2, Connector_JST:JST_XH_S3B-XH-A-1_1x03_P2.50mm_Horizontal
- removed J9: CAN_1, Connector_JST:JST_XH_S3B-XH-A-1_1x03_P2.50mm_Horizontal
- removed Q1: AO3401A, Package_TO_SOT_SMD:SOT-23
- removed R25, R26: 100k, PCM_Resistor_SMD_AKL:R_0603_1608Metric
- removed R53: 4.7k, PCM_Resistor_SMD_AKL:R_0603_1608Metric
- removed U7: TJA1051T, Package_SO:SOIC-8_3.9x4.9mm_P1.27mm
- added C20: 100nF, PCM_Capacitor_SMD_AKL:C_0603_1608Metric, F.Cu at (128.8, 85.7)
- added C24: 1uF, PCM_Capacitor_SMD_AKL:C_0603_1608Metric, F.Cu at (128.3, 102.9)
- added C25: 1uF, PCM_Capacitor_SMD_AKL:C_0603_1608Metric, F.Cu at (140.0, 103.0)
- added J2: Conn_01x08, Connector_JST:JST_VH_B8P-VH-B_1x08_P3.96mm_Vertical, B.Cu at (163.6, 122.8)
- added U5: SN65HVD230, Package_SO:SOIC-8_3.9x4.9mm_P1.27mm, F.Cu at (144.8, 106.0)
- C19: value 1uF -> 100nF
- C22: value 10uF -> 1uF
- R13, R3: value 100k -> 470k
- R14, R8: value 27k -> 82k
- R23, R38: value 1k -> 10k
- U4: value LIS3DH -> SN65HVD230; footprint Package_LGA:LGA-16_3x3mm_P0.5mm_LayoutBorder3x5y -> Package_SO:SOIC-8_3.9x4.9mm_P1.27mm
- U6: value TJA1051T -> LSM6DSL; footprint Package_SO:SOIC-8_3.9x4.9mm_P1.27mm -> Package_LGA:LGA-14_3x2.5mm_P0.5mm_LayoutBorder3x4y
- moved U4 24.0 mm to (133.0, 106.0), turned to -90 degrees
- moved U6 23.5 mm to (128.8, 82.8)
- moved C19 0.80 mm to (128.7, 79.9)
Connections:
- C48 pad 1: Net-(Q1-D) -> GND
- IC1 pad 24: /BATT_MEAS_ENA -> unconnected-(IC1-RXD0-Pad24)
- IC1 pad 6: /Rs_1 -> GND
- IC1 pad 9: /Rs_2 -> GND
- JP5 pad 1: IGN -> /IGN_SIG
- R8 pad 2: Net-(Q1-D) -> GND
- U4 pad 1: +3.3V -> /TXD_1
- U4 pad 2: unconnected-(U4-NC-Pad2) -> GND
- U4 pad 3: unconnected-(U4-NC-Pad3) -> +3.3V
- U4 pad 4: /SCL -> /RXD_1
- U4 pad 5: GND -> unconnected-(U4-Vref-Pad5)
- U4 pad 6: /SDA -> /CANL_1
- U4 pad 7: GND -> /CANH_1
- U4 pad 8: Net-(U4-CS) -> GND
- U6 pad 1: /TXD_1 -> GND
- U6 pad 3: +3.3V -> GND
- U6 pad 4: /RXD_1 -> /INT1
- U6 pad 5: unconnected-(U6-NC-Pad5) -> +3.3V
- U6 pad 6: /CANL_1 -> GND
- U6 pad 7: /CANH_1 -> GND
- U6 pad 8: /Rs_1 -> +3.3V
Routing:
- net GND: track 8.84 -> 59.5 mm, vias 0 -> 4
- net /Rs_1: track 31.4 -> 0.00 mm, vias 2 -> 0
- net /Rs_2: track 25.2 -> 0.00 mm, vias 2 -> 0
- net Net-(Q1-D): track 14.9 -> 0.00 mm, vias 2 -> 0
- net /IGN_SIG: track 11.2 -> 24.0 mm, vias 2 -> 4
- net /BATT_MEAS_ENA: track 12.0 -> 0.00 mm, vias 2 -> 0
- net +12V: track 55.4 -> 64.2 mm
- net IGN: track 56.9 -> 48.9 mm
- net +3.3V: track 18.7 -> 22.8 mm, vias 21 -> 23
- net /CANH_1: track 17.6 -> 21.5 mm
- net /CANL_1: track 19.1 -> 22.4 mm
- net /CANH_2: track 17.5 -> 20.1 mm
- net Net-(U4-CS): track 2.03 -> 0.00 mm
- net /CANL_2: track 19.2 -> 21.1 mm
- net /SCL: track 18.6 -> 19.2 mm
Other:
- board text added: "12"
- board text added: "ADCU-M"
- board text added: "CH1"
- board text added: "CH2"
- board text added: "CL1"
- board text added: "CL2"
- board text added: "IGN"
- board text added: "V1.0"
- board text removed: "ADCU-M v1.0"
- board text removed: "CAN1"
- board text removed: "CAN2"
- board text removed: "Irfan R"
- board text removed: "PWR"

Commit message: make prod files, clean up CAN wiring on slave
Parts:
- removed C11, C12, C13, C15, C16, C17, C18: 22uF, PCM_Capacitor_SMD_AKL:C_0603_1608Metric
- removed C14: 100nF, PCM_Capacitor_SMD_AKL:C_0603_1608Metric
- removed C4, C5, C6, C7, C8: 22nF, PCM_Capacitor_SMD_AKL:C_0603_1608Metric
- removed D2: SS54, PCM_JLCPCB:D_SMA
- removed JP1: SolderJumper_2_Bridged, Jumper:SolderJumper-2_P1.3mm_Bridged_Pad1.0x1.5mm
- removed JP5: SolderJumper_3_Open, Jumper:SolderJumper-3_P1.3mm_Open_RoundedPad1.0x1.5mm
- removed R10: 10k, PCM_Resistor_SMD_AKL:R_0805_2012Metric
- removed R11: 3.24k, PCM_Resistor_SMD_AKL:R_0805_2012Metric
- removed U3: AMS1117-3.3, Package_TO_SOT_SMD:SOT-223-3_TabPin2
- added C10: 220uF, Capacitor_THT:CP_Radial_D8.0mm_P3.50mm, F.Cu at (159.5, 106.2)
- added C26: 10uF, PCM_Capacitor_SMD_AKL:C_0603_1608Metric, F.Cu at (169.0, 86.2)
- added C34: 100nF, PCM_Capacitor_SMD_AKL:C_0603_1608Metric, F.Cu at (171.2, 102.5)
- added C35: 10uF, PCM_Capacitor_SMD_AKL:C_0603_1608Metric, F.Cu at (169.3, 102.5)
- added D1: B5819WS, PCM_JLCPCB:D_SOD-323, F.Cu at (135.8, 92.0)
- added D11: BAT54SW, Package_TO_SOT_SMD:SOT-323_SC-70, F.Cu at (166.8, 75.4)
- added D12: LED BLUE, PCM_LED_SMD_AKL:LED_0603_1608Metric, F.Cu at (166.1, 95.3)
- added D3: SS24FL, PCM_Diode_SMD_AKL:D_SOD-123F, F.Cu at (171.4, 106.5)
- added D5: BAT54SW, Package_TO_SOT_SMD:SOT-323_SC-70, F.Cu at (164.2, 75.4)
- added DZ2: BZT52C10S, PCM_Diode_SMD_AKL:D_SOD-323, F.Cu at (152.8, 112.6)
- added JP3: SolderJumper_2_Open, Jumper:SolderJumper-2_P1.3mm_Open_Pad1.0x1.5mm, F.Cu at (135.8, 95.4)
- added Q1: HL2309, PCM_Package_TO_SOT_SMD_AKL:SOT-23, F.Cu at (156.1, 112.5)
- added R16: 1k, PCM_Resistor_SMD_AKL:R_0603_1608Metric, F.Cu at (162.5, 98.3)
- added R17: 1k, PCM_Resistor_SMD_AKL:R_0603_1608Metric, F.Cu at (164.3, 98.3)
- added R18: 1k, PCM_Resistor_SMD_AKL:R_0603_1608Metric, F.Cu at (166.1, 98.3)
- added R19: 22, PCM_Resistor_SMD_AKL:R_0402_1005Metric, F.Cu at (138.2, 91.8)
- added R20: 22, PCM_Resistor_SMD_AKL:R_0402_1005Metric, F.Cu at (138.3, 93.0)
- added R21: 10k, PCM_Resistor_SMD_AKL:R_0603_1608Metric, F.Cu at (165.0, 111.8)
- added R22: 3.24k, PCM_Resistor_SMD_AKL:R_0603_1608Metric, F.Cu at (165.0, 113.5)
- added R39: 10k, PCM_Resistor_SMD_AKL:R_0603_1608Metric, F.Cu at (150.5, 112.8)
- added R40: 10k, PCM_Resistor_SMD_AKL:R_0603_1608Metric, F.Cu at (169.0, 89.8)
- added R41: 10k, PCM_Resistor_SMD_AKL:R_0603_1608Metric, F.Cu at (136.8, 89.5)
- added SW4: SW_SPST, Button_Switch_SMD:SW_SPST_TS-1088-xR025, F.Cu at (172.0, 88.0)
- D10, D9: value SS54 -> LED BLUE; footprint PCM_JLCPCB:D_SMA -> PCM_LED_SMD_AKL:LED_0603_1608Metric
- L1: footprint PCM_SparkFun-Coil:Inductor_7.3x6.6mm -> PCM_Inductor_SMD_AKL:L_Taiyo-Yuden_NR-40xx
- R13, R3: value 470k -> 430k
- R14: value 82k -> 83k
- R9: value 2k -> 4..7k
- moved D9 26.4 mm to (162.5, 95.3), turned to -90 degrees
- moved D10 19.3 mm to (164.3, 95.3), turned to -90 degrees
- moved C3 19.2 mm to (150.0, 106.1)
- moved L1 13.6 mm to (170.2, 97.5), turned to 0 degrees
- moved U2 11.6 mm to (170.3, 111.0), turned to 0 degrees
- moved D7 9.01 mm to (161.2, 111.8)
- moved R9 9.01 mm to (161.2, 113.5)
- moved C9 8.15 mm to (167.9, 106.1)
- moved H7 5.00 mm to (128.5, 117.5)
- moved H8 5.00 mm to (171.5, 117.5)
- moved J2 4.51 mm to (163.9, 118.2)
- moved R48 1.77 mm to (141.8, 109.5)
- moved U5 1.69 mm to (143.7, 104.8)
- moved C25 1.69 mm to (138.9, 101.8)
- moved C57 1.69 mm to (145.4, 109.5)
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Connections:
- C3 pad 1: Net-(JP5-B) -> +12V
- D10 pad 1: Net-(JP5-B) -> /LED2
- D10 pad 2: +12V -> Net-(D10-A)
- D9 pad 1: Net-(JP1-A) -> /LED1
- D9 pad 2: Net-(D9-Pad2) -> Net-(D9-A)
- IC1 pad 10: unconnected-(IC1-IO8-Pad10) -> Net-(IC1-IO8)
- IC1 pad 16: unconnected-(IC1-IO18-Pad16) -> /LED1
- IC1 pad 17: unconnected-(IC1-IO19-Pad17) -> /LED2
- IC1 pad 18: unconnected-(IC1-IO20-Pad18) -> /LED3
- IC1 pad 19: unconnected-(IC1-IO21-Pad19) -> Net-(IC1-IO21)
- IC1 pad 20: unconnected-(IC1-IO22-Pad20) -> /INT1
- IC1 pad 21: unconnected-(IC1-IO23-Pad21) -> /INT2
- IC1 pad 6: GND -> unconnected-(IC1-IO6-Pad6)
- IC1 pad 9: GND -> unconnected-(IC1-IO1-Pad9)
- J2 pad 3: +12V -> VIN
- J2 pad 8: unconnected-(J2-Pin_8-Pad8) -> GND
- J6 pad A4: Net-(D9-Pad2) -> Net-(D1-Pad2)
- J6 pad A6: /USB+ -> Net-(J6-D+-PadA6)
- J6 pad A7: /USB- -> Net-(J6-D--PadA7)
- J6 pad A9: Net-(D9-Pad2) -> Net-(D1-Pad2)
- J6 pad B4: Net-(D9-Pad2) -> Net-(D1-Pad2)
- J6 pad B6: /USB+ -> Net-(J6-D+-PadA6)
- J6 pad B7: /USB- -> Net-(J6-D--PadA7)
- J6 pad B9: Net-(D9-Pad2) -> Net-(D1-Pad2)
- L1 pad 2: +5V -> /Input Filtering/5V
- R13 pad 2: Net-(R13-Pad2) -> /IGN_SIG_PRE
- R14 pad 1: Net-(R13-Pad2) -> /IGN_SIG_PRE
- R15 pad 1: Net-(R13-Pad2) -> /IGN_SIG_PRE
- U2 pad 5: Net-(JP5-C) -> /IGN_SIG_PRE
- U2 pad 7: Net-(JP5-B) -> +12V
Routing:
- net +5V: track 57.0 -> 0.00 mm, vias 2 -> 0
- net GND: track 59.5 -> 7.12 mm, vias 4 -> 0
- net /INT2: track 0.00 -> 52.1 mm, vias 0 -> 2
- net /INT1: track 0.00 -> 47.5 mm, vias 0 -> 2
- net Net-(JP5-B): track 42.8 -> 0.00 mm, vias 6 -> 0
- net /IGN_SIG_PRE: track 0.00 -> 40.8 mm, vias 0 -> 2
- net +12V: track 64.2 -> 92.5 mm, vias 1 -> 5
- net /Input Filtering/5V: track 0.00 -> 23.0 mm, vias 0 -> 1
- net Net-(IC1-IO21): track 0.00 -> 17.5 mm
- net /USB+: track 15.8 -> 3.11 mm, vias 2 -> 0
- net Net-(J6-D+-PadA6): track 0.00 -> 11.6 mm, vias 0 -> 2
- net Net-(D9-Pad2): track 10.7 -> 0.00 mm, vias 2 -> 0
- net Net-(D1-Pad2): track 0.00 -> 10.6 mm, vias 0 -> 2
- net /IGN_SIG: track 24.0 -> 13.5 mm, vias 4 -> 2
- net Net-(JP5-C): track 10.2 -> 0.00 mm
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Other:
- board size 50 x 55 mm -> 50 x 50 mm
- board text added: "1"
- board text added: "2"
- board text added: "3"
- board text added: "RST"
- board text added: "USR"
