File: Master/Active-Damper-Master.kicad_sch (KiCad schematic)
At the start: 53 parts, among them IC1 ESP32-C6-WROOM-1-N8, J6 USB_C_Receptacle_USB2.0_16P, J7 POWER, J8 CAN_2, J9 CAN_1, Q1 AO3401A, SW2 SW_SPST, SW3 SW_SPST, U4 LIS3DH, U6 TJA1051T, U7 TJA1051T

Commit message: add prod files, not done
Parts:
- removed J7: POWER, Connector_JST:JST_XH_S3B-XH-A-1_1x03_P2.50mm_Horizontal, symbol Connector_Generic:Conn_01x03
- removed J8: CAN_2, Connector_JST:JST_XH_S3B-XH-A-1_1x03_P2.50mm_Horizontal, symbol Connector_Generic:Conn_01x03
- removed J9: CAN_1, Connector_JST:JST_XH_S3B-XH-A-1_1x03_P2.50mm_Horizontal, symbol Connector_Generic:Conn_01x03
- removed Q1: AO3401A, Package_TO_SOT_SMD:SOT-23, symbol Transistor_FET:AO3401A
- removed R25, R26: 100k, PCM_Resistor_SMD_AKL:R_0603_1608Metric, symbol Device:R
- removed R53: 4.7k, PCM_Resistor_SMD_AKL:R_0603_1608Metric, symbol Device:R
- removed U4: LIS3DH, Package_LGA:LGA-16_3x3mm_P0.5mm_LayoutBorder3x5y, symbol Sensor_Motion:LIS3DH
- removed U6, U7: TJA1051T, Package_SO:SOIC-8_3.9x4.9mm_P1.27mm, symbol Interface_CAN_LIN:TJA1051T
- added C20: 100nF, PCM_Capacitor_SMD_AKL:C_0603_1608Metric, symbol Device:C_Small
- added C24, C25: 1uF, PCM_Capacitor_SMD_AKL:C_0603_1608Metric, symbol Device:C_Small
- added J2: Conn_01x08, Connector_JST:JST_VH_B8P-VH-B_1x08_P3.96mm_Vertical, symbol Connector_Generic:Conn_01x08
- added U4, U5: SN65HVD230, Package_SO:SOIC-8_3.9x4.9mm_P1.27mm, symbol Interface_CAN_LIN:SN65HVD230
- added U6: LSM6DSL, Package_LGA:LGA-14_3x2.5mm_P0.5mm_LayoutBorder3x4y, symbol Sensor_Motion:LSM6DSL
- C19: value 1uF -> 100nF
- C22: value 10uF -> 1uF
- R13, R3: value 100k -> 470k
- R14, R8: value 27k -> 82k
- R23, R38: value 1k -> 10k
Connections:
- net Rs_1 is gone; now on net GND: IC1.6 (IO6)
- net Rs_2 is gone; now on net GND: IC1.9 (IO1)
- net +12V: now also J2.3 (Pin_3)
- net +3.3V: now also C20.2, C24.2, C25.2, U4.3 (VCC), U5.3 (VCC), U6.12 (CS), U6.5 (VDDIO), U6.8 (VDD)
- net CANH_1: now also J2.6 (Pin_6), U4.7 (CANH)
- net CANH_2: now also J2.4 (Pin_4), U5.7 (CANH)
- net CANL_1: now also J2.7 (Pin_7), U4.6 (CANL)
- net CANL_2: now also J2.5 (Pin_5), U5.6 (CANL)
- net GND: now also C48.1, R8.2, C20.1, C24.1, C25.1, J2.1 (Pin_1), U4.2 (GND), U4.8 (Rs), U5.2 (GND), U5.8 (Rs), U6.1 (SDO/SA0), U6.2 (SDX), U6.3 (SCX), U6.6 (GND), U6.7 (GND)
- net IGN: now also J2.2 (Pin_2)
- net INT1: now also U6.4 (INT1)
- net INT2: now also U6.9 (INT2)
- net RXD_1: now also U4.4 (R)
- net RXD_2: now also U5.4 (R)
- net SCL: now also U6.13 (SCL)
- net SDA: now also U6.14 (SDA)
- net TXD_1: now also U4.1 (D)
- net TXD_2: now also U5.1 (D)
- net BATT_MEAS_ENA: no longer names the net of IC1.24 (RXD0)
- no-connect marks 4 -> 13

Commit message: make prod files, clean up CAN wiring on slave
Parts:
- removed D9: SS54, PCM_JLCPCB:D_SMA, symbol PCM_JLCPCB-Diodes:Schottky,SS54
- removed JP1: SolderJumper_2_Bridged, Jumper:SolderJumper-2_P1.3mm_Bridged_Pad1.0x1.5mm, symbol Jumper:SolderJumper_2_Bridged
- added C26: 10uF, PCM_Capacitor_SMD_AKL:C_0603_1608Metric, symbol Device:C_Small
- added D1: B5819WS, PCM_JLCPCB:D_SOD-323, symbol JLCPCB-Diodes:Schottky,B5819WS
- added D10, D12, D9: LED BLUE, PCM_LED_SMD_AKL:LED_0603_1608Metric, symbol Device:LED
- added D11, D5: BAT54SW, Package_TO_SOT_SMD:SOT-323_SC-70, symbol Diode:BAT54SW
- added DZ2: BZT52C10S, PCM_Diode_SMD_AKL:D_SOD-323, symbol PCM_Diode_Zener_AKL:BZT52C10S
- added JP3: SolderJumper_2_Open, Jumper:SolderJumper-2_P1.3mm_Open_Pad1.0x1.5mm, symbol Jumper:SolderJumper_2_Open
- added Q1: HL2309, PCM_Package_TO_SOT_SMD_AKL:SOT-23, symbol JLCPCB-Transistors:PMOS,HL2309
- added R16, R17, R18: 1k, PCM_Resistor_SMD_AKL:R_0603_1608Metric, symbol Device:R
- added R19, R20: 22, PCM_Resistor_SMD_AKL:R_0402_1005Metric, symbol Device:R
- added R39, R40, R41: 10k, PCM_Resistor_SMD_AKL:R_0603_1608Metric, symbol Device:R
- added SW4: SW_SPST, Button_Switch_SMD:SW_SPST_TS-1088-xR025, symbol Switch:SW_SPST
- J2: KiLib_Generator (none) -> connector/JST
- R13, R3: value 470k -> 430k
- R14: value 82k -> 83k
- R9: value 2k -> 4..7k
- U4, U5: KiLib_Generator (none) -> package/gullwing
- U6: KiLib_Generator (none) -> package/no_lead
Connections:
- net +12V: now also DZ2.1 (K), JP3.2 (B), Q1.2 (S); no longer J2.3 (Pin_3)
- net +3.3V: now also D11.2 (K), D5.2 (K), R16.1, R17.1, R18.1, R40.2, R41.2
- net BATT_SIG: now also D5.3 (COM)
- net GND: now also J2.8 (Pin_8), C26.2, D11.1 (A), D5.1 (A), R39.1, SW4.2 (B); no longer IC1.6 (IO6), IC1.9 (IO1)
- net IGN_SIG: now also D11.3 (COM)
- net INT1: now also IC1.20 (IO22)
- net INT2: now also IC1.21 (IO23)
- net USB+: now also R20.2; no longer J6.A6 (D+), J6.B6 (D+)
- net USB-: now also R19.2; no longer J6.A7 (D-), J6.B7 (D-)
- net at IC1.10 (IO8): now also R41.1
- net LED1: now reaches IC1.16 (IO18)
- net LED1: now also D9.1 (K)
- net LED2: now reaches IC1.17 (IO19)
- net LED2: now also D10.1 (K)
- net LED3: now reaches IC1.18 (IO20)
- net LED3: now also D12.1 (K)
- net at IC1.19 (IO21): now also C26.1, R40.1, SW4.1 (A)
- net at J6.A4 (VBUS), J6.A9 (VBUS), J6.B4 (VBUS)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: now also D1.2
- net IGN_SIG_PRE: now reaches R13.2, R14.1, R15.1
- new net: D1.1, JP3.1 (A)
- new net: D12.2 (A), R18.2
- new net: DZ2.2 (A), Q1.1 (G), R39.2
- new net: J6.A6 (D+), J6.B6 (D+), R20.1
- new net: J6.A7 (D-), J6.B7 (D-), R19.1
- new net: D9.2 (A), R16.2
- new net: D10.2 (A), R17.2
- new net VIN: J2.3 (Pin_3), Q1.3 (D)
- no-connect marks 13 -> 7
Other:
- sheet Input Filtering ports: added EN; removed 5V, IGN
- moved on the sheet: J2
