File: Master/input.kicad_sch (KiCad schematic)
At the start: 23 parts, among them U2 TPS5430DDAR, U3 AMS1117-3.3

Commit message: make prod files, clean up CAN wiring on slave
Parts:
- removed C11, C12, C13, C15, C16, C17, C18: 22uF, PCM_Capacitor_SMD_AKL:C_0603_1608Metric, symbol Device:C_Small
- removed C14: 100nF, PCM_Capacitor_SMD_AKL:C_0603_1608Metric, symbol Device:C_Small
- removed C4, C5, C6, C7, C8: 22nF, PCM_Capacitor_SMD_AKL:C_0603_1608Metric, symbol Device:C_Small
- removed D10, D2: SS54, PCM_JLCPCB:D_SMA, symbol PCM_JLCPCB-Diodes:Schottky,SS54
- removed JP5: SolderJumper_3_Open, Jumper:SolderJumper-3_P1.3mm_Open_RoundedPad1.0x1.5mm, symbol Jumper:SolderJumper_3_Open
- removed R10: 10k, PCM_Resistor_SMD_AKL:R_0805_2012Metric, symbol PCM_Resistor_AKL:R_0805
- removed R11: 3.24k, PCM_Resistor_SMD_AKL:R_0805_2012Metric, symbol PCM_Resistor_AKL:R_0805
- removed U3: AMS1117-3.3, Package_TO_SOT_SMD:SOT-223-3_TabPin2, symbol Regulator_Linear:AMS1117-3.3
- added C10: 220uF, Capacitor_THT:CP_Radial_D8.0mm_P3.50mm, symbol Device:C_Polarized
- added C34: 100nF, PCM_Capacitor_SMD_AKL:C_0603_1608Metric, symbol Device:C_Small
- added C35: 10uF, PCM_Capacitor_SMD_AKL:C_0603_1608Metric, symbol Device:C_Small
- added D3: SS24FL, PCM_Diode_SMD_AKL:D_SOD-123F, symbol PCM_Diode_Schottky_AKL:SS24FL
- added R21: 10k, PCM_Resistor_SMD_AKL:R_0603_1608Metric, symbol PCM_Resistor_AKL:R_0805
- added R22: 3.24k, PCM_Resistor_SMD_AKL:R_0603_1608Metric, symbol PCM_Resistor_AKL:R_0805
- L1: footprint PCM_SparkFun-Coil:Inductor_7.3x6.6mm -> PCM_Inductor_SMD_AKL:L_Taiyo-Yuden_NR-40xx
Connections:
- net 5V: now also C10.1, R21.2
- net GND: now also C10.2, C34.1, C35.1, D3.2 (A), R22.1
- net VIN: now also C3.1, U2.7 (VIN), C34.2, C35.2
- net at C9.2, L1.1, U2.8 (PH): now also D3.1 (K)
- net EN: now reaches U2.5 (ENA)
- net at U2.4 (VSENSE): now also R21.1, R22.2
