File: Slave/Active-Damper-Slave.kicad_pcb (KiCad board)
At the start: 4 copper layers, 42.3 x 42.3 mm, 81 parts, among them IC2 AS5600-ASOM, IC3 ATA6563-GBQW1, IC4 ATA6563-GBQW1, J2 FL, J3 SHF-105-01-F-D-TH, J6 USB_C_Receptacle_USB2.0_16P, J7 POWER, J8 CAN_2, J9 CAN_1, SW1 SW_SPST, U1 STM32F103C8T6, U2 TPS5430DDAR, U3 AMS1117-3.3, U4 LIS3DH, U5 TMC2209-LA, X1 X50328MSB2GI

Commit message: add prod files, not done
Parts:
- removed C11, C12, C13, C15, C16, C17, C18: 22uF, PCM_Capacitor_SMD_AKL:C_0402_1005Metric
- removed C14: 100nF, PCM_Capacitor_SMD_AKL:C_0402_1005Metric
- removed C19: 1uF, PCM_Capacitor_SMD_AKL:C_0402_1005Metric
- removed C3: 220uF, Capacitor_THT:CP_Radial_D8.0mm_P3.50mm
- removed C4, C5, C6, C7, C8: 22nF, PCM_Capacitor_SMD_AKL:C_0603_1608Metric
- removed C57, C58: 100pF, PCM_Capacitor_SMD_AKL:C_0402_1005Metric
- removed C9: 10nF, PCM_Capacitor_SMD_AKL:C_0603_1608Metric
- removed D8: PESD1CAN, PCM_Package_TO_SOT_SMD_AKL:SOT-23
- removed IC4: ATA6563-GBQW1, SamacSys_Parts:SON65P300X300X90-9N-D
- removed J7: POWER, Connector_JST:JST_PH_S3B-PH-K_1x03_P2.00mm_Horizontal
- removed J8: CAN_2, Connector_JST:JST_PH_S3B-PH-K_1x03_P2.00mm_Horizontal
- removed J9: CAN_1, Connector_JST:JST_PH_S3B-PH-K_1x03_P2.00mm_Horizontal
- removed JP1: SolderJumper_2_Bridged, Jumper:SolderJumper-2_P1.3mm_Bridged_Pad1.0x1.5mm
- removed JP5: SolderJumper_3_Open, Jumper:SolderJumper-3_P1.3mm_Open_RoundedPad1.0x1.5mm
- removed L1: 15uH, PCM_SparkFun-Coil:Inductor_7.3x6.6mm
- removed R3: 100k, PCM_Resistor_SMD_AKL:R_0402_1005Metric
- removed R48, R49: 60, PCM_Capacitor_SMD_AKL:C_0603_1608Metric
- removed R51, R53, R54: 4.7k, PCM_Resistor_SMD_AKL:R_0402_1005Metric
- removed U2: TPS5430DDAR, PCM_JLCPCB:ESOP-8_L4.9-W3.9-P1.27-LS6.0-TL-EP
- removed U3: AMS1117-3.3, Package_TO_SOT_SMD:SOT-223-3_TabPin2
- removed U4: LIS3DH, Package_LGA:LGA-16_3x3mm_P0.5mm_LayoutBorder3x5y
- added C32: 22nF, PCM_Capacitor_SMD_AKL:C_0603_1608Metric, F.Cu at (157.5, 107.5)
- added C33: 22nF, PCM_Capacitor_SMD_AKL:C_0603_1608Metric, F.Cu at (157.5, 105.7)
- added C34: 22nF, PCM_Capacitor_SMD_AKL:C_0603_1608Metric, F.Cu at (157.5, 103.9)
- added C35: 22nF, PCM_Capacitor_SMD_AKL:C_0603_1608Metric, F.Cu at (157.5, 102.3)
- added C39: 100nF, PCM_Capacitor_SMD_AKL:C_0402_1005Metric, F.Cu at (136.0, 88.2)
- added C40: 100nF, PCM_Capacitor_SMD_AKL:C_0402_1005Metric, F.Cu at (137.0, 91.0)
- added C41: 0.1uF, PCM_Capacitor_SMD_AKL:C_0603_1608Metric, F.Cu at (160.2, 103.2)
- added C42: 22uF, PCM_Capacitor_SMD_AKL:C_0603_1608Metric, F.Cu at (159.5, 100.5)
- added IC1: LMR51610XFQDBVRQ1, SamacSys_Parts:SOT95P280X145-6N, F.Cu at (164.0, 106.4)
- added J4: FL, Connector_Wire:SolderWire-0.5sqmm_1x04_P4.6mm_D0.9mm_OD2.1mm, F.Cu at (133.5, 94.2)
- added J5: FL, Connector_Wire:SolderWire-0.5sqmm_1x04_P4.6mm_D0.9mm_OD2.1mm, F.Cu at (136.5, 94.2)
- added L2: 22uH, PCM_Inductor_SMD_AKL:L_Taiyo-Yuden_MD-4040, F.Cu at (163.8, 102.0)
- added R12: 100k, PCM_Resistor_SMD_AKL:R_0402_1005Metric, F.Cu at (123.8, 93.1)
- added R56: 4.7k, PCM_Resistor_SMD_AKL:R_0402_1005Metric, F.Cu at (139.0, 91.0)
- added R57: 4.7k, PCM_Resistor_SMD_AKL:R_0402_1005Metric, F.Cu at (138.0, 91.0)
- added R58: 10k, PCM_Resistor_SMD_AKL:R_0402_1005Metric, F.Cu at (154.0, 112.8)
- added R8: 69.8k, PCM_Resistor_SMD_AKL:R_0603_1608Metric, F.Cu at (159.8, 109.6)
- added R9: 22.1k, PCM_Resistor_SMD_AKL:R_0603_1608Metric, F.Cu at (160.2, 106.6)
- added U7: LSM6DSL, Package_LGA:LGA-14_3x2.5mm_P0.5mm_LayoutBorder3x4y, F.Cu at (134.6, 90.6)
- C21: value 1uF -> 220uF; footprint PCM_Capacitor_SMD_AKL:C_0402_1005Metric -> Capacitor_THT:CP_Radial_D8.0mm_P3.50mm
- C23: value 1uF -> 22nF; footprint PCM_Capacitor_SMD_AKL:C_0402_1005Metric -> PCM_Capacitor_SMD_AKL:C_0603_1608Metric
- D2: value SS54 -> B5819W SL; footprint PCM_JLCPCB:D_SMA -> PCM_JLCPCB:D_SOD-123
- IC3: value ATA6563-GBQW1 -> TCAN3413DRBR; footprint SamacSys_Parts:SON65P300X300X90-9N-D -> SamacSys_Parts:SON65P300X300X100-9N-D
- J2: footprint Connector_JST:JST_PH_S4B-PH-K_1x04_P2.00mm_Horizontal -> Connector_Wire:SolderWire-0.5sqmm_1x04_P4.6mm_D0.9mm_OD2.1mm
- JP3: footprint Jumper:SolderJumper-2_P1.3mm_Open_RoundedPad1.0x1.5mm -> Jumper:SolderJumper-2_P1.3mm_Open_Pad1.0x1.5mm; moved to F.Cu
- R10: value 10k -> 100k
- R11: value 3.24k -> 1.5k
- R4, R5: footprint PCM_Capacitor_SMD_AKL:C_2010_5025Metric_Pad1.52x2.65mm -> PCM_Resistor_SMD_AKL:R_2010_5025Metric; moved to F.Cu
- moved C23 38.0 mm to (163.8, 111.8)
- moved IC3 32.0 mm to (163.3, 96.0), turned to 180 degrees
- moved JP3 26.7 mm to (165.2, 90.7)
- moved C24 24.5 mm to (164.3, 98.7)
- moved C25 21.5 mm to (164.3, 93.7)
- moved C59 21.1 mm to (162.3, 98.7), turned to 180 degrees
- moved R4 20.0 mm to (160.2, 114.2), turned to -90 degrees
- moved C22 18.6 mm to (155.6, 112.2), turned to -90 degrees
- moved C30 17.8 mm to (157.2, 112.2), turned to -90 degrees
- moved C60 17.6 mm to (162.3, 93.7), turned to 180 degrees
- moved R52 17.1 mm to (159.5, 98.7), turned to 0 degrees
- moved R11 16.2 mm to (155.0, 93.5)
- moved C21 15.7 mm to (140.3, 106.8)
- moved D11 14.9 mm to (159.1, 96.0), turned to 180 degrees
- moved C31 14.5 mm to (153.0, 107.5), turned to -90 degrees
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Connections:
- C21 pad 1: GND -> +12V
- C21 pad 2: +3.3V -> GND
- C23 pad 2: +5V -> +12V
- C24 pad 1: GND -> +3.3V
- C24 pad 2: +5V -> GND
- C25 pad 1: GND -> +3.3V
- C25 pad 2: +3.3V -> GND
- D11 pad 1: /CANH_1 -> /CANL_1
- D11 pad 2: /CANL_1 -> /CANH_1
- D2 pad 2: GND -> +12V
- D5 pad 1: Net-(JP1-A) -> Net-(JP3-A)
- IC2 pad 8: /DIR -> /DIR_ENC
- IC3 pad 1: /TXD_2 -> /TXD_1
- IC3 pad 3: +5V -> +3.3V
- IC3 pad 4: /RXD_2 -> /RXD_1
- IC3 pad 6: /CANL_2 -> /CANL_1
- IC3 pad 7: /CANH_2 -> /CANH_1
- IC3 pad 8: /STBY_2 -> /STBY_1
- J2 pad 1: /BOUT2 -> /AOUT1
- J2 pad 2: /BOUT1 -> /AOUT2
- J2 pad 3: /AOUT2 -> /BOUT1
- J2 pad 4: /AOUT1 -> /BOUT2
- JP3 pad 2: Net-(JP3-B) -> +12V
- R10 pad 1: Net-(U2-VSENSE) -> +3.3V
- R10 pad 2: +5V -> /STBY_1
- R11 pad 1: GND -> /USB+
- R11 pad 2: Net-(U2-VSENSE) -> +3.3V
- U1 pad 10: /AIN1 -> /OUT
- U1 pad 11: /AIN2 -> unconnected-(U1-PA1-Pad11)
- U1 pad 12: /BIN1 -> unconnected-(U1-PA2-Pad12)
- U1 pad 13: /BIN2 -> unconnected-(U1-PA3-Pad13)
- U1 pad 16: unconnected-(U1-PA6-Pad16) -> /STDBY_DRV
- U1 pad 17: unconnected-(U1-PA7-Pad17) -> /DIR
- U1 pad 19: unconnected-(U1-PB1-Pad19) -> /STEP
- U1 pad 22: unconnected-(U1-PB11-Pad22) -> /~{EN}_DRV
- U1 pad 23: Net-(U1-VSS-Pad23) -> GND
- U1 pad 29: unconnected-(U1-PA8-Pad29) -> /STBY_1
- U1 pad 3: unconnected-(U1-PC14-Pad3) -> /DIR_ENC
- U1 pad 30: unconnected-(U1-PA9-Pad30) -> /~{PD}/UART
- U1 pad 35: Net-(U1-VSS-Pad23) -> GND
- U1 pad 39: unconnected-(U1-PB3-Pad39) -> /SWO/TDO
- U1 pad 45: unconnected-(U1-PB8-Pad45) -> /RXD_1
- U1 pad 46: unconnected-(U1-PB9-Pad46) -> /TXD_1
- U1 pad 47: Net-(U1-VSS-Pad23) -> GND
- U1 pad 8: unconnected-(U1-VSSA-Pad8) -> GND
- U5 pad 2: GND -> /~{EN}_DRV
- U5 pad 20: /STDBY -> /STDBY_DRV
Routing:
- net /CANH_1: track 0.00 -> 40.2 mm, vias 0 -> 1
- net /CANL_1: track 0.00 -> 39.5 mm, vias 0 -> 1
- net /SDA: track 0.00 -> 29.2 mm, vias 0 -> 3
- net /SCL: track 0.00 -> 28.0 mm, vias 0 -> 3
- net +3.3V: track 0.00 -> 28.0 mm, vias 0 -> 27
- net /~{RESET}: track 0.00 -> 24.7 mm, vias 0 -> 2
- net /SWDIO/TMS: track 0.00 -> 24.5 mm, vias 0 -> 1
- net /TXD_1: track 0.00 -> 22.4 mm, vias 0 -> 2
- net /RXD_1: track 0.00 -> 20.2 mm, vias 0 -> 2
- net /SWCLK/TCK: track 0.00 -> 18.9 mm, vias 0 -> 1
- net /SWO/TDO: track 0.00 -> 16.5 mm, vias 0 -> 1
- net /USB-: track 0.00 -> 15.8 mm
- net /USB+: track 0.00 -> 15.6 mm, vias 0 -> 2
- net Net-(U5-BRB): track 0.00 -> 13.8 mm, vias 0 -> 2
- net /~{PD}/UART: track 0.00 -> 13.1 mm, vias 0 -> 2
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- added copper zone on In1.Cu, net +12V
- removed copper zone on In2.Cu, net +12V
- removed copper zone on In2.Cu, net +5V
- removed copper zone on In1.Cu, net GND
Other:
- board size 42.3 x 42.3 mm -> 36.7 x 36.7 mm
- board text added: "12"
- board text added: "A1"
- board text added: "A2"
- board text added: "ADCU-S"
- board text added: "B1"
- board text added: "B2"
- board text added: "CH"
- board text added: "CL"
- board text added: "G"
- board text added: "V1.0"

Commit message: make prod files, clean up CAN wiring on slave
Parts:
- removed D11: PESD1CAN, PCM_Package_TO_SOT_SMD_AKL:SOT-23
- removed X1: X50328MSB2GI, PCM_JLCPCB:CRYSTAL-SMD_L5.0-W3.2
- added JP1: SolderJumper_2_Open, Jumper:SolderJumper-2_P1.3mm_Open_RoundedPad1.0x1.5mm, B.Cu at (159.4, 107.4)
- added JP5: SolderJumper_2_Open, Jumper:SolderJumper-2_P1.3mm_Open_RoundedPad1.0x1.5mm, B.Cu at (159.4, 104.9)
- added JP6: SolderJumper_2_Open, Jumper:SolderJumper-2_P1.3mm_Open_RoundedPad1.0x1.5mm, B.Cu at (159.4, 102.4)
- added ye1: X50328MSB2GI, PCM_JLCPCB:CRYSTAL-SMD_L5.0-W3.2, F.Cu at (140.1, 98.9)
- JP4: footprint Jumper:SolderJumper-2_P1.3mm_Open_RoundedPad1.0x1.5mm -> Jumper:SolderJumper-2_P1.3mm_Open_Pad1.0x1.5mm
- R1: value 1k -> 10k
- moved R12 20.4 mm to (143.8, 97.2), turned to -90 degrees
Connections:
- U1 pad 26: unconnected-(U1-PB13-Pad26) -> Net-(JP1-B)
- U1 pad 27: unconnected-(U1-PB14-Pad27) -> Net-(JP5-B)
- U1 pad 28: unconnected-(U1-PB15-Pad28) -> Net-(JP6-B)
Routing:
- net /STDBY_DRV: track 1.44 -> 9.85 mm
- net Net-(JP1-B): track 0.00 -> 7.96 mm, vias 0 -> 1
- net Net-(JP5-B): track 0.00 -> 6.91 mm, vias 0 -> 1
- net Net-(JP6-B): track 0.00 -> 5.52 mm, vias 0 -> 1
- net /CANH_1: track 40.2 -> 36.4 mm
- net /DIR_ENC: track 1.52 -> 3.42 mm
- net +3.3V: track 28.0 -> 29.4 mm
Other:
- board text added: "1"
- board text added: "2"
- board text added: "3"
- board text added: "TERM"
