File: Slave/Active-Damper-Slave.kicad_sch (KiCad schematic)
At the start: 4 parts, among them IC2 AS5600-ASOM

Commit message: keep working on slave
Parts:
- removed R50: 4.7k, PCM_Resistor_SMD_AKL:R_0402_1005Metric, symbol Device:R
- added C1, C26: 100nF, PCM_Capacitor_SMD_AKL:C_0402_1005Metric, symbol Device:C_Small
- added C10, C28: 10uF, PCM_Capacitor_SMD_AKL:C_0402_1005Metric, symbol Device:C_Small
- added C19, C21, C23, C24, C25, C27: 1uF, PCM_Capacitor_SMD_AKL:C_0402_1005Metric, symbol Device:C_Small
- added C2, C29: 22pF, PCM_Capacitor_SMD_AKL:C_0402_1005Metric, symbol Device:C_Small
- added C22, C30: 22nF, PCM_Capacitor_SMD_AKL:C_0603_1608Metric, symbol Device:C_Small
- added C31: 2.2uF, PCM_Capacitor_SMD_AKL:C_0402_1005Metric, symbol Device:C_Small
- added C57, C58, C59, C60: 100pF, PCM_Capacitor_SMD_AKL:C_0402_1005Metric, symbol Device:C_Small
- added D11, D8: PESD1CAN, PCM_Package_TO_SOT_SMD_AKL:SOT-23, symbol PCM_Diode_TVS_AKL:PESD1CAN
- added D5: B5819WS, PCM_JLCPCB:D_SOD-323, symbol JLCPCB-Diodes:Schottky,B5819WS
- added H5, H6, H7, H8: MountingHole, MountingHole:MountingHole_3.2mm_M3_ISO14580_Pad_TopBottom, symbol Mechanical:MountingHole_Pad
- added IC3, IC4: ATA6563-GBQW1, SamacSys_Parts:SON65P300X300X90-9N-D, symbol SamacSys_Parts:ATA6563-GBQW1
- added J1: Conn_ARM_JTAG_SWD_10, PCM_SparkFun-Connector:2x05_P1.27mm, symbol Connector:Conn_ARM_JTAG_SWD_10
- added J2: FL, Connector_JST:JST_PH_S4B-PH-K_1x04_P2.00mm_Horizontal, symbol Connector_Generic:Conn_01x04
- added J3: SHF-105-01-F-D-TH, SamacSys_Parts:SHF10501FDTH, symbol SamacSys_Parts:SHF-105-01-F-D-TH
- added J6: USB_C_Receptacle_USB2.0_16P, Connector_USB:USB_C_Receptacle_HRO_TYPE-C-31-M-12, symbol Connector:USB_C_Receptacle_USB2.0_16P
- added J7: POWER, Connector_JST:JST_PH_S3B-PH-K_1x03_P2.00mm_Horizontal, symbol Connector_Generic:Conn_01x03
- added J8: CAN_2, Connector_JST:JST_PH_S3B-PH-K_1x03_P2.00mm_Horizontal, symbol Connector_Generic:Conn_01x03
- added J9: CAN_1, Connector_JST:JST_PH_S3B-PH-K_1x03_P2.00mm_Horizontal, symbol Connector_Generic:Conn_01x03
- added JP1: SolderJumper_2_Bridged, Jumper:SolderJumper-2_P1.3mm_Bridged_Pad1.0x1.5mm, symbol Jumper:SolderJumper_2_Bridged
- added JP3, JP4: SolderJumper_2_Open, Jumper:SolderJumper-2_P1.3mm_Open_RoundedPad1.0x1.5mm, symbol Jumper:SolderJumper_2_Open
- added R1: 1k, PCM_Resistor_SMD_AKL:R_0402_1005Metric, symbol Device:R
- added R2: 10k, PCM_Resistor_SMD_AKL:R_0402_1005Metric, symbol Device:R_Small
- added R3: 100k, PCM_Resistor_SMD_AKL:R_0402_1005Metric, symbol Device:R
- added R4, R5: 0.1, PCM_Capacitor_SMD_AKL:C_2010_5025Metric_Pad1.52x2.65mm, symbol Device:R
- added R48, R49, R52, R55: 60, PCM_Capacitor_SMD_AKL:C_0603_1608Metric, symbol Device:R
- added R51, R53, R54: 4.7k, PCM_Resistor_SMD_AKL:R_0402_1005Metric, symbol Device:R
- added R6, R7: 5k1, PCM_Resistor_SMD_AKL:R_0603_1608Metric, symbol Device:R
- added SW1: SW_SPST, Button_Switch_SMD:SW_SPST_TS-1088-xR025, symbol Switch:SW_SPST
- added U1: STM32F103C8T6, PCM_JLCPCB:LQFP-48_7x7mm_P0.5mm, symbol JLCPCB-MCUs:STM32F103C8T6
- added U4: LIS3DH, Package_LGA:LGA-16_3x3mm_P0.5mm_LayoutBorder3x5y, symbol Sensor_Motion:LIS3DH
- added U5: TMC2209-LA, Package_DFN_QFN:VQFN-28-1EP_5x5mm_P0.5mm_EP3.7x3.7mm_ThermalVias, symbol Driver_Motor:TMC2209-LA
- added X1: X50328MSB2GI, PCM_JLCPCB:CRYSTAL-SMD_L5.0-W3.2, symbol PCM_JLCPCB-Crystals:Crystal, 8MHz, 20pF, ±10ppm
- C20: footprint PCM_Capacitor_SMD_AKL:C_0603_1608Metric -> PCM_Capacitor_SMD_AKL:C_0402_1005Metric
- IC2: footprint SOIC127P600X175-8N -> SamacSys_Parts:SOIC127P600X175-8N
Connections:
- net +3.3V: now also C10.2, C19.2, C21.2, C25.2, C26.2, C27.2, C28.2, IC3.5 (VIO), IC4.5 (VIO), J1.1 (VTref), J3.1, R1.1, R51.2, R53.2, R54.2, U1.1 (VBAT), U1.24 (VDD), U1.36 (VDD), U1.48 (VDD), U1.9 (VDDA), U4.1 (VDD_IO), U4.14 (VDD), U5.15 (VCC_IO)
- net DIR: now also U5.19 (DIR)
- net GND: now also C1.1, C10.1, C19.1, C2.1, C21.1, C23.1, C24.1, C25.1, C26.1, C27.1, C28.1, C29.1, C31.1, C57.2, C58.1, C59.2, C60.1, D11.3 (Com), D8.3 (Com), H5.1, H6.1, H7.1, H8.1, IC3.2 (GND), IC3.9 (EP), IC4.2 (GND), IC4.9 (EP), J1.3 (GND), J1.5 (GND), J1.9 (GNDDetect), J3.3, J3.9, J6.A1 (GND), J6.A12 (GND), J6.A8 (SBU1), J6.B1 (GND), J6.B12 (GND), J6.B8 (SBU2), J6.SH (SHIELD), J7.1 (Pin_1), J8.3 (Pin_3), J9.3 (Pin_3), R2.1, R3.2, R4.2, R5.2, R6.2, R7.2, SW1.2 (B), U4.10 (GND), U4.12 (GND), U4.13 (ADC3), U4.15 (ADC2), U4.16 (ADC1), U4.5 (GND), U4.7 (SDO), U5.10 (MS2/AD1), U5.11 (DIAG), U5.12 (INDEX), U5.13 (CLK), U5.18 (GND), U5.2 (~{EN}), U5.25 (NC), U5.29 (GND), U5.3 (GND), U5.7 (SPREAD), U5.9 (MS1/AD0)
- net SCL: now also R54.1, U1.42 (PB6), U4.4 (SPC)
- net SDA: now also R51.1, U1.43 (PB7), U4.6 (SDI)
- net OUT: now reaches IC2.3 (OUT)
- new net: JP3.1 (A), R49.2
- new net: JP3.2 (B), R48.1
- new net: D5.1, JP1.1 (A)
- new net: D5.2, J6.A4 (VBUS), J6.A9 (VBUS), J6.B4 (VBUS), J6.B9 (VBUS)
- new net: R53.1, U4.8 (CS)
- new net: JP4.1 (A), R55.2
- new net: C31.2, U5.8 (5VOUT)
- new net: C30.1, U5.6 (VCP)
- new net: J6.A5 (CC1), R6.1
- new net: C29.2, U1.6 (PD1), X1.1
- new net: R5.1, U5.23 (BRA)
- new net: R4.1, U5.27 (BRB)
- new net: C22.2, U5.4 (CPO)
- new net: C22.1, U5.5 (CPI)
- new net: J6.B5 (CC2), R7.1
- new net: R2.2, U1.44 (BOOT0)
- new net: JP4.2 (B), R52.1
- new net: C2.2, U1.5 (PD0), X1.2
- new net: U1.23 (VSS), U1.35 (VSS), U1.47 (VSS)
- new net +12V: C30.2, J7.3 (Pin_3), U5.22 (VS), U5.28 (VS)
- new net +5V: C23.2, C24.2, IC3.3 (VCC), IC4.3 (VCC), JP1.2 (B)
- new net AIN1: U1.10 (PA0)
- new net AIN2: U1.11 (PA1)
- new net AOUT1: J2.4 (Pin_4), U5.24 (OA1)
- new net AOUT2: J2.3 (Pin_3), U5.21 (OA2)
- new net BIN1: U1.12 (PA2)
- new net BIN2: U1.13 (PA3)
- new net BOUT1: J2.2 (Pin_2), U5.26 (OB1)
- new net BOUT2: J2.1 (Pin_1), U5.1 (OB2)
- new net CANH_1: C59.1, D11.1 (A1), IC4.7 (CANH), J9.2 (Pin_2), R52.2
- new net CANH_2: C57.1, D8.1 (A1), IC3.7 (CANH), J8.2 (Pin_2), R48.2
- new net CANL_1: C60.2, D11.2 (A2), IC4.6 (CANL), J9.1 (Pin_1), R55.1
- new net CANL_2: C58.2, D8.2 (A2), IC3.6 (CANL), J8.1 (Pin_1), R49.1
- new net IGN: J7.2 (Pin_2)
- new net INT1: U4.11 (INT1)
- new net INT2: U4.9 (INT2)
- new net RXD_1: IC4.4 (RXD)
- new net RXD_2: IC3.4 (RXD)
- new net STBY_1: IC4.8 (STBY)
- new net STBY_2: IC3.8 (STBY)
- new net STDBY: R3.1, U5.20 (STDBY)
- new net STEP: U5.16 (STEP)
- new net SWCLK/TCK: J1.4 (SWCLK/TCK), J3.4, U1.37 (PA14)
- new net SWDIO/TMS: J1.2 (SWDIO/TMS), J3.2, U1.34 (PA13)
- new net SWO/TDO: J1.6 (SWO/TDO), J3.6
- new net TXD_1: IC4.1 (TXD)
- new net TXD_2: IC3.1 (TXD)
- new net USB+: J6.A6 (D+), J6.B6 (D+), U1.33 (PA12)
- new net USB-: J6.A7 (D-), J6.B7 (D-), U1.32 (PA11)
- new net ~{PD}/UART: U5.14 (~{PD}/UART)
- new net ~{RESET}: C1.2, J1.10 (~{RESET}), J3.10, R1.2, SW1.1 (A), U1.7 (NRST)
- no-connect marks 0 -> 5
Other:
- added sheet Input Filtering (input.kicad_sch)
- note added: "CAN"
- note added: "Connector"
- note added: "IMU"
- note added: "Mounting"
- note added: "Power"
- note added: "USB"
- note added: "VMEAS"

Commit message: add prod files, not done
Parts:
- removed C19, C21, C23: 1uF, PCM_Capacitor_SMD_AKL:C_0402_1005Metric, symbol Device:C_Small
- removed C57, C58: 100pF, PCM_Capacitor_SMD_AKL:C_0402_1005Metric, symbol Device:C_Small
- removed D8: PESD1CAN, PCM_Package_TO_SOT_SMD_AKL:SOT-23, symbol PCM_Diode_TVS_AKL:PESD1CAN
- removed IC3, IC4: ATA6563-GBQW1, SamacSys_Parts:SON65P300X300X90-9N-D, symbol SamacSys_Parts:ATA6563-GBQW1
- removed J7: POWER, Connector_JST:JST_PH_S3B-PH-K_1x03_P2.00mm_Horizontal, symbol Connector_Generic:Conn_01x03
- removed J8: CAN_2, Connector_JST:JST_PH_S3B-PH-K_1x03_P2.00mm_Horizontal, symbol Connector_Generic:Conn_01x03
- removed J9: CAN_1, Connector_JST:JST_PH_S3B-PH-K_1x03_P2.00mm_Horizontal, symbol Connector_Generic:Conn_01x03
- removed JP1: SolderJumper_2_Bridged, Jumper:SolderJumper-2_P1.3mm_Bridged_Pad1.0x1.5mm, symbol Jumper:SolderJumper_2_Bridged
- removed R3: 100k, PCM_Resistor_SMD_AKL:R_0402_1005Metric, symbol Device:R
- removed R48, R49: 60, PCM_Capacitor_SMD_AKL:C_0603_1608Metric, symbol Device:R
- removed R51, R53, R54: 4.7k, PCM_Resistor_SMD_AKL:R_0402_1005Metric, symbol Device:R
- removed U4: LIS3DH, Package_LGA:LGA-16_3x3mm_P0.5mm_LayoutBorder3x5y, symbol Sensor_Motion:LIS3DH
- added C39, C40: 100nF, PCM_Capacitor_SMD_AKL:C_0402_1005Metric, symbol Device:C_Small
- added IC3: TCAN3413DRBR, SamacSys_Parts:SON65P300X300X100-9N-D, symbol SamacSys_Parts:TCAN3413DRBR
- added J4, J5: FL, Connector_Wire:SolderWire-0.5sqmm_1x04_P4.6mm_D0.9mm_OD2.1mm, symbol Connector_Generic:Conn_01x04
- added R10, R12: 100k, PCM_Resistor_SMD_AKL:R_0402_1005Metric, symbol Device:R
- added R11: 1.5k, PCM_Resistor_SMD_AKL:R_0603_1608Metric, symbol Device:R
- added R56, R57: 4.7k, PCM_Resistor_SMD_AKL:R_0402_1005Metric, symbol Device:R
- added R58: 10k, PCM_Resistor_SMD_AKL:R_0402_1005Metric, symbol Device:R
- added U7: LSM6DSL, Package_LGA:LGA-14_3x2.5mm_P0.5mm_LayoutBorder3x4y, symbol Sensor_Motion:LSM6DSL
- J2: footprint Connector_JST:JST_PH_S4B-PH-K_1x04_P2.00mm_Horizontal -> Connector_Wire:SolderWire-0.5sqmm_1x04_P4.6mm_D0.9mm_OD2.1mm; KiLib_Generator (none) -> connector/JST
- JP3: footprint Jumper:SolderJumper-2_P1.3mm_Open_RoundedPad1.0x1.5mm -> Jumper:SolderJumper-2_P1.3mm_Open_Pad1.0x1.5mm
- R4, R5: footprint PCM_Capacitor_SMD_AKL:C_2010_5025Metric_Pad1.52x2.65mm -> PCM_Resistor_SMD_AKL:R_2010_5025Metric
- U5: KiLib_Generator (none) -> package/no_lead; LCSC (none) -> C2150710
Connections:
- net +5V is gone; now on net GND: C24.2
- net AIN1 is gone; now on net OUT: U1.10 (PA0)
- net STDBY is gone; now on net STDBY_DRV: U5.20 (STDBY)
- net +12V: now also JP3.2 (B), J4.4 (Pin_4), J5.4 (Pin_4)
- net +3.3V: now also C24.1, C25.1, C39.2, C40.2, IC3.3 (VCC), IC3.5 (SHDNVIO), R10.1, R11.2, R12.1, R56.2, R57.2, R58.2, U7.12 (CS), U7.5 (VDDIO), U7.8 (VDD); no longer C25.2
- net AOUT1: now also J2.1 (Pin_1); no longer J2.4 (Pin_4)
- net AOUT2: now also J2.2 (Pin_2); no longer J2.3 (Pin_3)
- net BOUT1: now also J2.3 (Pin_3); no longer J2.2 (Pin_2)
- net BOUT2: now also J2.4 (Pin_4); no longer J2.1 (Pin_1)
- net CANH_1: now also D11.2 (A2), IC3.7 (CANH), J4.1 (Pin_1), J5.1 (Pin_1); no longer D11.1 (A1)
- net CANL_1: now also D11.1 (A1), IC3.6 (CANL), J4.2 (Pin_2), J5.2 (Pin_2); no longer D11.2 (A2)
- net DIR: now also U1.17 (PA7); no longer IC2.8 (DIR)
- net GND: now also C25.2, U1.23 (VSS), U1.35 (VSS), U1.47 (VSS), U1.8 (VSSA), C39.1, C40.1, IC3.2 (GND), IC3.9 (EP), J4.3 (Pin_3), J5.3 (Pin_3), U7.1 (SDO/SA0), U7.2 (SDX), U7.3 (SCX), U7.6 (GND), U7.7 (GND); no longer C24.1, C25.1, U5.2 (~{EN})
- net INT1: now also U7.4 (INT1)
- net INT2: now also U7.9 (INT2)
- net RXD_1: now also U1.45 (PB8), IC3.4 (RXD)
- net SCL: now also R56.1, U7.13 (SCL)
- net SDA: now also R57.1, U7.14 (SDA)
- net STBY_1: now also U1.29 (PA8), IC3.8 (STB), R10.2
- net STEP: now also U1.19 (PB1)
- net SWO/TDO: now also U1.39 (PB3)
- net TXD_1: now also U1.46 (PB9), IC3.1 (TXD)
- net USB+: now also R11.1
- net ~{PD}/UART: now also U1.30 (PA9)
- net at JP3.1 (A): now also D5.1
- net STDBY_DRV: now reaches U1.16 (PA6)
- net ~{EN}_DRV: now reaches U1.22 (PB11)
- net ~{EN}_DRV: now also U5.2 (~{EN}), R58.1
- net DIR_ENC: now reaches U1.3 (PC14)
- net DIR_ENC: now also IC2.8 (DIR), R12.2
- net AIN2: no longer names the net of U1.11 (PA1)
- net BIN1: no longer names the net of U1.12 (PA2)
- net BIN2: no longer names the net of U1.13 (PA3)
Other:
- sheet Input Filtering ports: added none; removed 5V, IGN
- note removed: "IMU"
- moved on the sheet: U5

Commit message: make prod files, clean up CAN wiring on slave
Parts:
- removed D11: PESD1CAN, PCM_Package_TO_SOT_SMD_AKL:SOT-23, symbol PCM_Diode_TVS_AKL:PESD1CAN
- added JP1, JP5, JP6: SolderJumper_2_Open, Jumper:SolderJumper-2_P1.3mm_Open_RoundedPad1.0x1.5mm, symbol Jumper:SolderJumper_2_Open
- J1: footprint PCM_SparkFun-Connector:2x05_P1.27mm -> SamacSys_Parts:SHF10501FDTH; now fitted
- JP4: footprint Jumper:SolderJumper-2_P1.3mm_Open_RoundedPad1.0x1.5mm -> Jumper:SolderJumper-2_P1.3mm_Open_Pad1.0x1.5mm
- R1: value 1k -> 10k
- renumbered X1 to ye1
Connections:
- net GND: now also JP1.1 (A), JP5.1 (A), JP6.1 (A)
- net at U1.26 (PB13): now also JP1.2 (B)
- net at U1.27 (PB14): now also JP5.2 (B)
- net at U1.28 (PB15): now also JP6.2 (B)
- no-connect marks 5 -> 20
Other:
- moved on the sheet: C1, C10, C26, C27, C28, J2, J4, J5, SW1, U1, U5
