File: Daughter/imu_daughter_board/imu_daughter_board.kicad_sch (KiCad schematic)
At the start: 4 parts, among them J1 Conn_01x04, U1 STM32F030C8T6, U2 LSM6DSL, U3 SN65HVD230DR

Commit message: almost done schem_daughter
Parts:
- removed U1: STM32F030C8T6, PCM_JLCPCB:LQFP-48_7x7mm_P0.5mm, symbol PCM_JLCPCB-MCUs:STM32F030C8T6
- removed U3: SN65HVD230DR, PCM_JLCPCB:SOIC-8_L4.9-W3.9-P1.27-LS6.0-BL, symbol PCM_JLCPCB-Interface:Transceiver, CAN, SN65HVD230DR
- added C1, C12, C2, C5, C6, C7, C8, C9: 100n, PCM_SparkFun-Resistor:R_0402_1005Metric, symbol Device:C
- added C10, C11: 8.2n, PCM_SparkFun-Resistor:R_0402_1005Metric, symbol Device:C
- added C3, C4: 100p, PCM_SparkFun-Resistor:R_0402_1005Metric, symbol Device:C
- added IC1: TCAN3413DRBR, SamacSys_Parts:SON65P300X300X100-9N-D, symbol SamacSys_Parts:TCAN3413DRBR
- added JP1, JP2, JP3, JP4: SolderJumper_2_Open, Jumper:SolderJumper-2_P1.3mm_Open_Pad1.0x1.5mm, symbol Jumper:SolderJumper_2_Open
- added R1, R10, R2, R3, R4, R7, R8, R9: 10k, PCM_SparkFun-Resistor:R_0402_1005Metric, symbol Device:R
- added R5, R6: 120, PCM_Resistor_SMD_AKL:R_0402_1005Metric, symbol Device:R
- added SW1: SW_SPST, Button_Switch_SMD:SW_SPST_TS-1088-xR025, symbol Switch:SW_SPST
- added U1: STM32F103C8Tx, Package_QFP:LQFP-48_7x7mm_P0.5mm, symbol MCU_ST_STM32F1:STM32F103C8Tx
- added X1: SMD3225-4, PCM_Crystal_AKL:Crystal_SMD_3225-4Pin_3.2x2.5mm, symbol PCM_Crystal_AKL:SMD3225-4
- J1: footprint Connector_JST:JST_PH_S4B-PH-K_1x04_P2.00mm_Horizontal -> Connector_Wire:SolderWire-0.5sqmm_1x04_P4.6mm_D0.9mm_OD2.1mm; KiLib_Generator (none) -> connector/JST
- U2: KiLib_Generator (none) -> package/no_lead
Connections:
- net at U2.1 (SDO/SA0): now also R2.2
- net at U2.12 (CS): now also R1.2
- net SCL: now reaches U2.13 (SCL)
- net SCL: now also R3.2, U1.42 (PB6)
- net SDA: now reaches U2.14 (SDA)
- net SDA: now also R4.2, U1.43 (PB7)
- net GND: now reaches U2.2 (SDX)
- net GND: now also J1.4 (Pin_4), U2.3 (SCX), U2.6 (GND), U2.7 (GND), C1.1, C10.1, C11.2, C12.1, C2.2, C3.2, C4.1, C5.1, C6.1, C7.2, C8.1, C9.2, IC1.2 (GND), IC1.9 (EP), JP2.1 (A), JP3.1 (A), JP4.1 (A), R10.1, R8.2, SW1.1 (A), U1.23 (VSS), U1.35 (VSS), U1.47 (VSS), U1.8 (VSSA), X1.2, X1.4
- net INT1: now reaches U2.4 (INT1)
- net INT1: now also U1.40 (PB4)
- net 3.3V: now reaches U2.5 (VDDIO)
- net 3.3V: now also U2.8 (VDD), C1.2, C2.1, C5.2, C6.2, C7.1, C8.2, C9.1, IC1.3 (VCC), R1.1, R2.1, R3.1, R4.1, R7.1, R9.1, U1.24 (VDD), U1.36 (VDD), U1.48 (VDD), U1.9 (VDDA)
- net INT2: now reaches U2.9 (INT2)
- net INT2: now also U1.41 (PB5)
- net +12V: now reaches J1.1 (Pin_1)
- net CAN_H: now reaches J1.2 (Pin_2)
- net CAN_H: now also C4.2, IC1.7 (CANH), R5.1
- net CAN_L: now reaches J1.3 (Pin_3)
- net CAN_L: now also C3.1, IC1.6 (CANL), R6.2
- new net: JP2.2 (B), U1.15 (PA5)
- new net: JP1.2 (B), R5.2
- new net: JP4.2 (B), U1.13 (PA3)
- new net: JP3.2 (B), U1.14 (PA4)
- new net: R10.2, U1.44 (BOOT0)
- new net: C12.2, R9.2, SW1.2 (B), U1.7 (NRST)
- new net: JP1.1 (A), R6.1
- new net RCC_H: C11.1, U1.5 (PD0), X1.1
- new net RCC_L: C10.2, U1.6 (PD1), X1.3
- new net RXD: IC1.4 (RXD), U1.32 (PA11)
- new net SHDNVIO: IC1.5 (SHDNVIO), R8.1, U1.30 (PA9)
- new net STB: IC1.8 (STB), R7.2, U1.31 (PA10)
- new net SWCLK: U1.37 (PA14)
- new net SWDIO: U1.34 (PA13)
- new net SWO: U1.39 (PB3)
- new net TXD: IC1.1 (TXD), U1.33 (PA12)
- no-connect marks 0 -> 22
Other:
- note added: "CL1 = CL2 = 2 X (CL - 5pF) = 2 X (9pF-5pF) = 8pF"
- moved on the sheet: J1, U2

Commit message: sch done
Parts:
- added C13: 10u, PCM_Capacitor_SMD_AKL:C_0603_1608Metric_Pad1.05x0.95mm, symbol Device:C
- added C14: 10n, PCM_Capacitor_SMD_AKL:C_0603_1608Metric_Pad1.05x0.95mm, symbol Device:C
- added C16: 6TPE220MAP, 2R5TAE330MF, symbol SamacSys_Parts:6TPE220MAP
- added D1: SS14F, PCM_Diode_SMD_AKL:D_SMAFL, symbol PCM_Diode_Schottky_AKL:SS14F
- added DZ1: BZT52C10S, PCM_Diode_SMD_AKL:D_SOD-323, symbol PCM_Diode_Zener_AKL:BZT52C10S
- added J2: Conn_ARM_JTAG_SWD_10, SamacSys_Parts:SHF10501FDTH, symbol Connector:Conn_ARM_JTAG_SWD_10
- added L1: 27u, PCM_Inductor_SMD_AKL:L_Taiyo-Yuden_MD-4040, symbol Device:L
- added Q1: HL2309, PCM_JLCPCB:Q_SOT-23, symbol PCM_JLCPCB-Transistors:PMOS,HL2309
- added R11, R13: 10k, PCM_Resistor_SMD_AKL:R_0603_1608Metric, symbol Device:R
- added R12: 5.9k, PCM_Resistor_SMD_AKL:R_0603_1608Metric, symbol Device:R
- added U3: TPS5430DDA, Package_SO:TI_SO-PowerPAD-8_ThermalVias, symbol Regulator_Switching:TPS5430DDA
- C1, C10, C11, C12, C2, C3, C4, C5, C6, C7, C8, C9, R1, R10, R2, R3, R4, R7, R8, R9: footprint PCM_SparkFun-Resistor:R_0402_1005Metric -> PCM_Capacitor_SMD_AKL:C_0402_1005Metric
Connections:
- net +12V: now also C13.1, DZ1.1 (K), Q1.2 (S), U3.7 (VIN); no longer J1.1 (Pin_1)
- net 3.3V: now also C16.1 (+), J2.1 (VTref), L1.2, R11.1
- net GND: now also C13.2, C16.2 (-), D1.2 (A), J2.3 (GND), J2.5 (GND), J2.9 (GNDDetect), R12.2, R13.2, U3.6 (GND), U3.9 (GNDPAD)
- net SWCLK: now also J2.4 (SWCLK/TCK)
- net SWDIO: now also J2.2 (SWDIO/TMS)
- net SWO: now also J2.6 (SWO/TDO)
- net RST: now reaches C12.2, R9.2, SW1.2 (B), U1.7 (NRST)
- net RST: now also J2.10 (~{RESET})
- net CAN_H renamed CANP
- net CAN_L renamed CANN
- new net: C14.1, U3.1 (BOOT)
- new net: R11.2, R12.1, U3.4 (VSENSE)
- new net: C14.2, D1.1 (K), L1.1, U3.8 (PH)
- new net: DZ1.2 (A), Q1.1 (G), R13.1
- new net VIN: J1.1 (Pin_1), Q1.3 (D)
- no-connect marks 22 -> 25
Other:
- note added: "-50℃~+150℃ 3A 40V 500uA@40V 550mV@3A Independent SMA(DO-214AC) Schottky Diodes ROHS"
- note added: "10mV = (250mA *0.25)/(Cbulk*500khz) + (250mA * ESR max)"
- note added: "Diode stops energy from disspating to ground"
- note added: "FNR4020S270MT"
- note added: "Ideal"
- note added: "Iout = 250mA"
- note added: "L_min= 3.310 * (12 - 3.3) / (12 * K_ind * 500khz) Using K_ind of 0.2, Lmin = =0.0000239975 = \approx 24uH 24 µH is an E24 preferred value, but 22 µH and 27 µH are more common for power inductors."
- note added: "Maybe not important yet"
- note added: "R2 = R1 * 1.221 / (3.3 - 1.221) R1 = 10kohm R2 = 10e3 * 1.221 / (3.3 - 1.221) 5873.01587302"
- note added: "Sus"
- note added: "This Range may not function properly"
- note added: "Use 5.90 kΩ, 1%-it's a standard E96 value closest to your calculated 5.873 kΩ."
- note added: "V_delta = 10mV"
- note added: "Vpp max = 20mV"
- note added: "fsw = 500khz"

Commit message: review daughter
Parts:
- R3, R4: value 10k -> 4.7k
- R5, R6: value 120 -> 60
Connections:
- no-connect marks 25 -> 24
Other:
- note added: "BUCK"
- note added: "CAN _Tranceiver"
- note added: "CONN"
- note added: "MCU"
- note added: "REVPROT"
- note added: "Sensor"
- moved on the sheet: C1, C2, C5, R1, R10, SW1
