File: Daughter/imu_daughter_board/imu_daughter_board.kicad_pcb (KiCad board)
At the start: 2 copper layers, 3 parts, among them J1 Conn_01x04, U1 STM32F030C8T6, U2 LSM6DSL

Commit message: almost done schem_daughter
Parts:
- added C1: 100n, PCM_SparkFun-Resistor:R_0402_1005Metric, F.Cu at (97.0, 80.5)
- added D1: PESD2CAN, PCM_Package_TO_SOT_SMD_AKL:SOT-23, F.Cu at (150.7, 94.2)
- added IC1: TCAN3413DRBR, SamacSys_Parts:SON65P300X300X100-9N-D, F.Cu at (145.7, 94.2)
- added R1: 10k, PCM_SparkFun-Resistor:R_0402_1005Metric, F.Cu at (154.5, 92.8)
- added R1: 10k, PCM_JLCPCB:R_0402, F.Cu at (89.0, 75.5)
- added R2: 10k, PCM_SparkFun-Resistor:R_0402_1005Metric, F.Cu at (102.5, 81.5)
- U1: value STM32F030C8T6 -> STM32F103C8Tx; footprint PCM_JLCPCB:LQFP-48_7x7mm_P0.5mm -> Package_QFP:LQFP-48_7x7mm_P0.5mm
- moved U1 49.4 mm to (148.7, 86.2)
Connections:
- U1 pad 32: unconnected-(U1-PA11-Pad32) -> /RXD
- U1 pad 33: unconnected-(U1-PA12-Pad33) -> /TXD
- U1 pad 35: unconnected-(U1-PF6-Pad35) -> Net-(U1-VSS-Pad23)
- U1 pad 40: unconnected-(U1-PB4-Pad40) -> /INT1
- U1 pad 41: unconnected-(U1-PB5-Pad41) -> /INT2
- U1 pad 42: unconnected-(U1-PB6-Pad42) -> /SCL
- U1 pad 43: unconnected-(U1-PB7-Pad43) -> /SDA
- U2 pad 1: unconnected-(U2-SDO/SA0-Pad1) -> Net-(U2-SDO/SA0)
- U2 pad 12: unconnected-(U2-CS-Pad12) -> Net-(U2-CS)
- U2 pad 13: unconnected-(U2-SCL-Pad13) -> /SCL
- U2 pad 14: unconnected-(U2-SDA-Pad14) -> /SDA
- U2 pad 2: unconnected-(U2-SDX-Pad2) -> /GND
- U2 pad 3: unconnected-(U2-SCX-Pad3) -> /GND
- U2 pad 4: unconnected-(U2-INT1-Pad4) -> /INT1
- U2 pad 6: Net-(U2-GND-Pad6) -> /GND
- U2 pad 7: Net-(U2-GND-Pad6) -> /GND
- U2 pad 9: unconnected-(U2-INT2-Pad9) -> /INT2

Commit message: sch done
Parts:
- added C10: 8.2n, PCM_Capacitor_SMD_AKL:C_0402_1005Metric, F.Cu at (126.3, 74.5)
- added C11: 8.2n, PCM_Capacitor_SMD_AKL:C_0402_1005Metric, F.Cu at (126.3, 64.0)
- added C12: 100n, PCM_Capacitor_SMD_AKL:C_0402_1005Metric, F.Cu at (112.1, 83.7)
- added C13: 10u, PCM_Capacitor_SMD_AKL:C_0603_1608Metric_Pad1.05x0.95mm, F.Cu at (202.1, 79.1)
- added C14: 10n, PCM_Capacitor_SMD_AKL:C_0603_1608Metric_Pad1.05x0.95mm, F.Cu at (160.4, 83.3)
- added C15: C_Polarized, Capacitor_THT:CP_Radial_D8.0mm_P3.50mm, F.Cu at (149.6, 88.7)
- added C2: 100n, PCM_Capacitor_SMD_AKL:C_0402_1005Metric, F.Cu at (145.2, 56.4)
- added C3: 100p, PCM_Capacitor_SMD_AKL:C_0402_1005Metric, F.Cu at (133.7, 109.0)
- added C4: 100p, PCM_Capacitor_SMD_AKL:C_0402_1005Metric, F.Cu at (140.2, 107.0)
- added C5: 100n, PCM_Capacitor_SMD_AKL:C_0402_1005Metric, F.Cu at (145.5, 75.3)
- added C6: 100n, PCM_Capacitor_SMD_AKL:C_0402_1005Metric, F.Cu at (143.3, 70.8)
- added C7: 100n, PCM_Capacitor_SMD_AKL:C_0402_1005Metric, F.Cu at (139.3, 80.3)
- added C8: 100n, PCM_Capacitor_SMD_AKL:C_0402_1005Metric, F.Cu at (129.8, 74.3)
- added C9: 100n, PCM_Capacitor_SMD_AKL:C_0402_1005Metric, F.Cu at (134.3, 67.3)
- added DZ1: BZT52C10S, PCM_Diode_SMD_AKL:D_SOD-323, F.Cu at (162.4, 77.8)
- added J2: Conn_ARM_JTAG_SWD_10, SamacSys_Parts:SHF10501FDTH, F.Cu at (145.7, 65.8)
- added JP1: SolderJumper_2_Open, Jumper:SolderJumper-2_P1.3mm_Open_Pad1.0x1.5mm, F.Cu at (136.5, 114.0)
- added JP2: SolderJumper_2_Open, Jumper:SolderJumper-2_P1.3mm_Open_Pad1.0x1.5mm, F.Cu at (125.7, 87.2)
- added JP3: SolderJumper_2_Open, Jumper:SolderJumper-2_P1.3mm_Open_Pad1.0x1.5mm, F.Cu at (129.5, 84.7)
- added JP4: SolderJumper_2_Open, Jumper:SolderJumper-2_P1.3mm_Open_Pad1.0x1.5mm, F.Cu at (133.3, 83.4)
- added L1: 27u, PCM_Inductor_SMD_AKL:L_Taiyo-Yuden_MD-4040, F.Cu at (151.5, 82.5)
- added Q1: HL2309, PCM_JLCPCB:Q_SOT-23, F.Cu at (161.9, 74.3)
- added R10: 10k, PCM_Capacitor_SMD_AKL:C_0402_1005Metric, F.Cu at (116.3, 84.8)
- added R11: 10k, PCM_Resistor_SMD_AKL:R_0603_1608Metric, F.Cu at (168.4, 88.1)
- added R12: 5.9k, PCM_Resistor_SMD_AKL:R_0603_1608Metric, F.Cu at (168.4, 84.3)
- added R13: 10k, PCM_Resistor_SMD_AKL:R_0603_1608Metric, F.Cu at (158.6, 77.8)
- added R3: 10k, PCM_Capacitor_SMD_AKL:C_0402_1005Metric, F.Cu at (135.8, 59.8)
- added R4: 10k, PCM_Capacitor_SMD_AKL:C_0402_1005Metric, F.Cu at (135.3, 55.8)
- added R5: 120, PCM_Resistor_SMD_AKL:R_0402_1005Metric, F.Cu at (139.1, 109.6)
- added R6: 120, PCM_Resistor_SMD_AKL:R_0402_1005Metric, F.Cu at (136.7, 109.6)
- added R7: 10k, PCM_Capacitor_SMD_AKL:C_0402_1005Metric, F.Cu at (138.6, 105.5)
- added R8: 10k, PCM_Capacitor_SMD_AKL:C_0402_1005Metric, F.Cu at (135.7, 105.5)
- added R9: 10k, PCM_Capacitor_SMD_AKL:C_0402_1005Metric, F.Cu at (120.1, 74.2)
- added SW1: SW_SPST, Button_Switch_SMD:SW_SPST_TS-1088-xR025, F.Cu at (113.5, 79.3)
- added U3: TPS5430DDA, Package_SO:TI_SO-PowerPAD-8_ThermalVias, F.Cu at (164.2, 83.4)
- added X1: SMD3225-4, PCM_Crystal_AKL:Crystal_SMD_3225-4Pin_3.2x2.5mm, F.Cu at (126.3, 69.8)
- C1, R1, R2: footprint PCM_SparkFun-Resistor:R_0402_1005Metric -> PCM_Capacitor_SMD_AKL:C_0402_1005Metric
- D1: value PESD2CAN -> SS14F; footprint PCM_Package_TO_SOT_SMD_AKL:SOT-23 -> PCM_Diode_SMD_AKL:D_SMAFL
- J1: footprint Connector_JST:JST_PH_S4B-PH-K_1x04_P2.00mm_Horizontal -> Connector_Wire:SolderWire-0.5sqmm_1x04_P4.6mm_D0.9mm_OD2.1mm
- moved J1 71.1 mm to (168.0, 69.9), turned to 90 degrees
- moved C1 50.1 mm to (139.1, 53.4), turned to 180 degrees
- moved R1 47.4 mm to (132.8, 57.3)
- moved R2 44.3 mm to (135.8, 52.3)
- moved R1 41.7 mm to (132.8, 57.3)
- moved U2 36.7 mm to (139.6, 57.5)
- moved U1 17.5 mm to (136.7, 73.4)
- moved D1 12.0 mm to (157.0, 84.0), turned to -90 degrees
- moved IC1 9.43 mm to (139.7, 101.5), turned to -90 degrees
Connections:
- C1 pad 1: unconnected-(C1-Pad1) -> GND
- C1 pad 2: unconnected-(C1-Pad2) -> 3.3V
- D1 pad 1: unconnected-(D1-A1-Pad1) -> Net-(D1-K)
- D1 pad 2: unconnected-(D1-A2-Pad2) -> GND
- IC1 pad 1: unconnected-(IC1-TXD-Pad1) -> /TXD
- IC1 pad 2: unconnected-(IC1-GND-Pad2) -> GND
- IC1 pad 3: unconnected-(IC1-VCC-Pad3) -> 3.3V
- IC1 pad 4: unconnected-(IC1-RXD-Pad4) -> /RXD
- IC1 pad 5: unconnected-(IC1-SHDNVIO-Pad5) -> /SHDNVIO
- IC1 pad 6: unconnected-(IC1-CANL-Pad6) -> /CANN
- IC1 pad 7: unconnected-(IC1-CANH-Pad7) -> /CANP
- IC1 pad 8: unconnected-(IC1-STB-Pad8) -> /STB
- IC1 pad 9: unconnected-(IC1-EP-Pad9) -> GND
- J1 pad 1: unconnected-(J1-Pin_1-Pad1) -> VIN
- J1 pad 2: unconnected-(J1-Pin_2-Pad2) -> /CANP
- J1 pad 3: unconnected-(J1-Pin_3-Pad3) -> /CANN
- J1 pad 4: unconnected-(J1-Pin_4-Pad4) -> GND
- R1 pad 1: /3V3 -> 3.3V
- R2 pad 1: /3V3 -> 3.3V
- U1 pad 13: unconnected-(U1-PA3-Pad13) -> Net-(JP4-B)
- U1 pad 14: unconnected-(U1-PA4-Pad14) -> Net-(JP3-B)
- U1 pad 15: unconnected-(U1-PA5-Pad15) -> Net-(JP2-B)
- U1 pad 23: Net-(U1-VSS-Pad23) -> GND
- U1 pad 24: unconnected-(U1-VDD-Pad24) -> 3.3V
- U1 pad 30: unconnected-(U1-PA9-Pad30) -> /SHDNVIO
- U1 pad 31: unconnected-(U1-PA10-Pad31) -> /STB
- U1 pad 34: unconnected-(U1-PA13-Pad34) -> /SWDIO
- U1 pad 35: Net-(U1-VSS-Pad23) -> GND
- U1 pad 36: unconnected-(U1-VDD-Pad36) -> 3.3V
- U1 pad 37: unconnected-(U1-PA14-Pad37) -> /SWCLK
- U1 pad 39: unconnected-(U1-PB3-Pad39) -> /SWO
- U1 pad 44: unconnected-(U1-BOOT0-Pad44) -> Net-(U1-BOOT0)
- U1 pad 47: Net-(U1-VSS-Pad23) -> GND
- U1 pad 48: unconnected-(U1-VDD-Pad48) -> 3.3V
- U1 pad 5: unconnected-(U1-PD0-Pad5) -> /RCC_H
- U1 pad 6: unconnected-(U1-PD1-Pad6) -> /RCC_L
- U1 pad 7: unconnected-(U1-NRST-Pad7) -> /RST
- U1 pad 8: unconnected-(U1-VSSA-Pad8) -> GND
- U1 pad 9: unconnected-(U1-VDDA-Pad9) -> 3.3V
- U2 pad 2: /GND -> GND
- U2 pad 3: /GND -> GND
- U2 pad 5: unconnected-(U2-VDDIO-Pad5) -> 3.3V
- U2 pad 6: /GND -> GND
- U2 pad 7: /GND -> GND
- U2 pad 8: unconnected-(U2-VDD-Pad8) -> 3.3V
Routing:
- net 3.3V: track 0.00 -> 5.99 mm
- net Net-(DZ1-A): track 0.00 -> 5.97 mm
- net +12V: track 0.00 -> 5.76 mm
- net Net-(D1-K): track 0.00 -> 5.37 mm
- net Net-(U3-VSENSE): track 0.00 -> 4.55 mm
- net Net-(U3-BOOT): track 0.00 -> 3.45 mm
- net VIN: track 0.00 -> 2.06 mm
Other:
- board text added: "Main Sheet"

Commit message: review daughter
Parts:
- removed C15: C_Polarized, Capacitor_THT:CP_Radial_D8.0mm_P3.50mm
- R3, R4: value 10k -> 4.7k
- R5, R6: value 120 -> 60
- moved R5 87.1 mm to (222.2, 83.3)
- moved R6 87.1 mm to (219.7, 83.3)
- moved C1 87.1 mm to (222.1, 27.1)
- moved JP1 87.1 mm to (219.6, 87.8)
- moved R13 87.1 mm to (241.6, 51.5)
- moved IC1 87.1 mm to (222.7, 75.3)
- moved R9 87.1 mm to (203.2, 48.0)
- moved C3 87.1 mm to (216.7, 82.8)
- moved C4 87.1 mm to (223.2, 80.8)
- moved R8 87.1 mm to (218.7, 79.3)
- moved R1 87.1 mm to (215.8, 31.0) (x2)
- moved R2 87.1 mm to (218.8, 26.0)
- moved R3 87.1 mm to (218.8, 33.5)
- moved R4 87.1 mm to (218.3, 29.5)
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Other:
- board outline added: 40 x 20 mm

Commit message: draft 1 complete
Parts:
- removed the R1 at (215.8, 31.0)
- added C16: 6TPE220MAP, SamacSys_Parts:2R5TAE330MF, F.Cu at (153.0, 100.1)
- J1, JP2, JP3, JP4: moved to B.Cu
- moved C13 129.9 mm to (167.0, 106.6), turned to -90 degrees
- moved R12 111.9 mm to (149.5, 104.1), turned to 180 degrees
- moved C2 111.1 mm to (144.5, 103.1)
- moved R11 107.6 mm to (152.5, 104.1), turned to 180 degrees
- moved C5 107.3 mm to (138.5, 107.5), turned to -90 degrees
- moved R2 107.2 mm to (142.2, 101.0), turned to 90 degrees
- moved C9 106.4 mm to (132.0, 104.6), turned to -90 degrees
- moved C1 106.1 mm to (147.0, 102.1), turned to 90 degrees
- moved U2 104.8 mm to (144.5, 101.1)
- moved C6 104.4 mm to (134.8, 94.6), turned to 0 degrees
- moved R4 100.8 mm to (144.5, 98.1), turned to 180 degrees
- moved R3 98.4 mm to (145.5, 99.1), turned to 180 degrees
- moved U3 98.3 mm to (162.0, 106.1), turned to 0 degrees
- moved D1 97.2 mm to (156.0, 106.6)
- moved L1 97.2 mm to (152.0, 107.6), turned to 90 degrees
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Routing:
- net GND: track 0.00 -> 42.2 mm, vias 0 -> 31
- net /SWO: track 0.00 -> 35.8 mm, vias 0 -> 1
- net /CANP: track 0.00 -> 31.5 mm, vias 0 -> 2
- net /CANN: track 0.00 -> 31.5 mm, vias 0 -> 2
- net /RST: track 0.00 -> 31.1 mm, vias 0 -> 2
- net /SWCLK: track 0.00 -> 28.8 mm, vias 0 -> 1
- net /INT2: track 0.00 -> 11.3 mm, vias 0 -> 2
- net /SHDNVIO: track 0.00 -> 11.2 mm
- net Net-(JP4-B): track 0.00 -> 10.7 mm, vias 0 -> 1
- net Net-(JP3-B): track 0.00 -> 10.6 mm, vias 0 -> 1
- net /RCC_L: track 0.00 -> 10.4 mm
- net /STB: track 0.00 -> 10.1 mm
- net Net-(JP2-B): track 0.00 -> 9.04 mm, vias 0 -> 1
- net Net-(U3-VSENSE): track 4.55 -> 12.0 mm
- net Net-(D1-K): track 5.37 -> 12.1 mm, vias 0 -> 2
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- added copper zone on F.Cu, net 3.3V
- added copper zone on B.Cu, net GND
Other:
- board size 40 x 20 mm -> 41.5 x 20 mm

Commit message: needs checking
Routing:
- net /SWDIO: track 0.00 -> 30.2 mm, vias 0 -> 3
- net /SCL: track 1.57 -> 11.1 mm, vias 0 -> 2
- net /SDA: track 0.00 -> 8.38 mm, vias 0 -> 2
- net Net-(D1-K): track 12.1 -> 18.8 mm, vias 2 -> 3
- net Net-(U2-CS): track 0.00 -> 2.29 mm
- net GND: track 42.2 -> 44.1 mm, vias 31 -> 33
- net VIN: track 8.22 -> 9.92 mm
- net /CANP: track 31.5 -> 31.0 mm
- net /CANN: track 31.5 -> 30.9 mm
- net /RXD: track 6.18 -> 5.63 mm, vias 0 -> 2
- net /TXD: track 3.32 -> 3.82 mm
- net /STB: track 10.1 -> 9.64 mm, vias 0 -> 2
- net /SHDNVIO: track 11.2 -> 11.3 mm, vias 0 -> 2
- net /RST: vias 2 -> 4

Commit message: done needs review, all the errors are all related to footprint or pink overlap looks good in 3d
Parts:
- removed R1: 10k, PCM_Capacitor_SMD_AKL:C_0402_1005Metric
- J1: moved to F.Cu
- JP1: moved to B.Cu
- moved C9 104.0 mm to (228.2, 65.2), turned to 0 degrees
- moved C5 100.1 mm to (230.0, 67.0)
- moved R12 98.1 mm to (242.5, 72.8), turned to -90 degrees
- moved R11 97.0 mm to (244.2, 72.8), turned to 90 degrees
- moved IC1 96.1 mm to (230.2, 70.2), turned to -90 degrees
- moved R7 96.0 mm to (232.8, 69.2), turned to -90 degrees
- moved L1 94.3 mm to (235.8, 64.2), turned to -90 degrees
- moved JP2 93.0 mm to (224.5, 72.5)
- moved R5 93.0 mm to (233.0, 73.2)
- moved R13 92.9 mm to (241.5, 57.0)
- moved D1 92.6 mm to (235.8, 59.5), turned to 180 degrees
- moved U1 92.6 mm to (223.5, 69.0), turned to 0 degrees
- moved C4 92.5 mm to (231.2, 73.2), turned to 180 degrees
- moved R6 92.3 mm to (232.2, 75.5), turned to 180 degrees
- moved R8 92.1 mm to (228.2, 73.2), turned to -90 degrees
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Connections:
- U2 pad 12: Net-(U2-CS) -> 3.3V
Routing:
- net /SWO: track 35.8 -> 5.50 mm, vias 1 -> 0
- net /SWCLK: track 28.8 -> 5.72 mm, vias 1 -> 0
- net /SWDIO: track 30.2 -> 9.44 mm, vias 3 -> 1
- net /INT1: track 5.98 -> 18.8 mm
- net /INT2: track 11.4 -> 21.2 mm
- net Net-(D1-K): track 18.8 -> 9.25 mm, vias 3 -> 0
- net Net-(U3-VSENSE): track 12.0 -> 3.54 mm
- net VIN: track 9.92 -> 2.35 mm, vias 1 -> 0
- net Net-(JP3-B): track 10.6 -> 3.35 mm
- net /STB: track 9.64 -> 16.7 mm
- net Net-(JP4-B): track 10.7 -> 3.97 mm
- net Net-(U1-BOOT0): track 2.87 -> 9.48 mm
- net /SHDNVIO: track 11.3 -> 5.47 mm, vias 2 -> 0
- net Net-(U2-SDO/SA0): track 1.14 -> 6.84 mm, vias 0 -> 2
- net /CANP: track 31.0 -> 26.4 mm, vias 2 -> 1
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Other:
- board size 41.5 x 20 mm -> 37.8 x 21 mm
- board text removed: "Main Sheet"

Commit message: ready to source
Routing:
- net GND: track 48.5 -> 46.1 mm
- net /CANP: track 26.4 -> 24.6 mm
- net /CANN: track 28.5 -> 27.7 mm
- net /RST: track 32.4 -> 31.7 mm
- net /RCC_L: track 7.54 -> 7.01 mm
Other:
- board size 37.8 x 21 mm -> 38.5 x 21 mm
