File: Daughter/imu_daughter_board backup/imu_daughter_board.kicad_sch (KiCad schematic)
At the start: 43 parts, among them IC1 TCAN3413DRBR, J1 Conn_01x04, J2 Conn_ARM_JTAG_SWD_10, Q1 HL2309, SW1 SW_SPST, U1 STM32F103C8Tx, U2 LSM6DSL, U3 TPS5430DDA, X1 SMD3225-4

Commit message: done needs review, all the errors are all related to footprint or pink overlap looks good in 3d
Parts:
- added R1: 10k, PCM_Capacitor_SMD_AKL:C_0402_1005Metric, symbol Device:R
Connections:
- net 3.3V: now also R1.1; no longer U2.12 (CS)
- new net: R1.2, U2.12 (CS)
- no-connect marks 25 -> 24
Changed lines of the file:
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@@
 	)
 	(no_connect
-		(at 185.42 116.84)
-	)
-	(no_connect
 		(at 92.71 135.89)
 	)
@@
 	(wire
 		(pts
-			(xy 22.86 49.53) (xy 22.86 62.23)
-		)
-		(stroke
-			(width 0)
-			(type default)
-		)
-	)
-	(wire
-		(pts
 			(xy 57.15 46.99) (xy 46.99 46.99)
 		)
@@
 	(wire
 		(pts
+			(xy 22.86 57.15) (xy 22.86 62.23)
+		)
+		(stroke
+			(width 0)
+			(type default)
+		)
+	)
+	(wire
+		(pts
 			(xy 173.99 102.87) (xy 173.99 106.68)
 		)
@@
 			(justify left bottom)
 		)
-		(property "Netclass" "CAN"
+		(property "Net Class" "CAN"
 			(at 210.82 59.69 0)
 			(show_name no)
@@
 			(justify left bottom)
 		)
-		(property "Netclass" "CAN"
+		(property "Net Class" "CAN"
 			(at 209.55 38.1 0)
 			(show_name no)
@@
 			(justify right bottom)
 		)
-		(property "Netclass" "CAN"
+		(property "Net Class" "CAN"
 			(at 234.95 29.21 0)
 			(show_name no)
@@
 			(justify right bottom)
 		)
-		(property "Netclass" "CAN"
+		(property "Net Class" "CAN"
 			(at 234.95 34.29 0)
 			(show_name no)
@@
 					(unit 1)
 				)
+			)
+		)
+	)
+	(symbol
+		(lib_id "Device:R")
+		(at 22.86 53.34 0)
+		(unit 1)
+		(body_style 1)
+		(exclude_from_sim no)
+		(in_bom yes)
+		(on_board yes)
+		(in_pos_files yes)
+		(dnp no)
+		(fields_autoplaced yes)
+		(property "Reference" "R1"
+			(at 25.4 52.0699 0)
+			(show_name no)
+			(do_not_autoplace no)
+			(effects
+				(font
+					(size 1.27 1.27)
+				)
+				(justify left)
+			)
+		)
+		(property "Value" "10k"
+			(at 25.4 54.6099 0)
+			(show_name no)
+			(do_not_autoplace no)
+			(effects
+				(font
+					(size 1.27 1.27)
+				)
+				(justify left)
+			)
+		)
+		(property "Footprint" "PCM_Capacitor_SMD_AKL:C_0402_1005Metric"
+			(at 21.082 53.34 90)
+			(hide yes)
+			(show_name no)
+			(do_not_autoplace no)
+			(effects
+				(font
+					(size 1.27 1.27)
+				)
+			)
+		)
+		(property "Datasheet" ""
+			(at 22.86 53.34 0)
+			(hide yes)
+			(show_name no)
+			(do_not_autoplace no)
+			(effects
+				(font
+					(size 1.27 1.27)
+				)
+			)
+		)
+		(property "Description" ""
+			(at 22.86 53.34 0)
+			(hide yes)
+			(show_name no)
+			(do_not_autoplace no)
+			(effects
+				(font
+					(size 1.27 1.27)
+				)
+			)
+		)
+		(pin "1"
+		)
+		(pin "2"
+		)
+		(instances
+			(project "imu_daughter_board"
+				(path "/6be3c0d3-4a91-4db5-bca9-cbf66493484f"
+					(reference "R1")
+					(unit 1)
+				)
